File: hardware/mule/mule.kicad_sch (KiCad schematic)
At the start: 65 parts, among them J1 IDC-40 task-PC event bus, J2 IDC-40 Pi event bus, J3 BARCODE_OUT test points, J4 Isolated-domain outputs, J5 Opto spare 1 bench injection, J6 Opto spare 2 bench injection, J7 ISO_5V/ISO_GND test point, J8 +5V DC in, U1 SN74LVC541APW, U2 SN74LVC541APW, U3 SN74LVC541APW, U4 SN74HCT541PW, U5 PC847, U6 TMA-0505S, U7 LD1117S33TR

Commit message: fix(hw): bidirectional clamp, logic-output optos, real Pi GPIO map
Coordinator fix round 1 on the mule schematic (hardware/gen/gen_mule.py):

- Input clamp is now genuinely bidirectional. BAV99 (previous choice) is
  common-anode and cannot clamp one signal to two rails with both diodes
  doing correct-direction work; switched to Diode:BAT54S, whose pin 3
  ("COM") is a real series midpoint, wired signal->COM, DGND->anode,
  +3V3->cathode. Flags a residual concern for bring-up: the lower
  Schottky forward drop means the high-side diode now conducts on every
  normal 5V logic-high, not just a fault, sinking current into +3V3.

- Optocoupler is now logic (open-collector) output, not phototransistor,
  so propagation-delay/edge-quality bring-up measurements (checks 5-6)
  validate the same part class the main board actually uses. Switched
  Isolator:PC847 -> two Isolator:HCPL-4661 packages. Correction flagged
  rather than silently applied: HCPL-4661 is 2-channel, not quad as
  described (confirmed against distributor listings and its 8-pin DIP
  pin budget) -- two packages, same part, not a vendor/output-type swap.

- Pi-side header (J2) now presents EVT_D0_PI..EVT_D15_PI and
  EVT_STROBE_PI at their real Raspberry Pi 40-pin physical positions
  (GPIO0-15 data, GPIO16 strobe; cross-checked against gpiozero's pin
  table), not sequential numbering, so the bring-up PIO capture test
  (check 7) can actually run. GPIO0/GPIO1 get an added 330R series
  resistor between buffer and header pin (boot-time I2C HAT-ID probe
  contention, same technique and value as the plan's Task 9 Step 2),
  with an on-sheet text note about config.txt's force_eeprom_read=0.
  BARCODE_PI also moved to its real GPIO17 position. Task-PC side (J1)
  stays sequential per the coordinator's own call.

- hardware/gen/check_mule_netlist.py extended to assert the GPIO
  mapping against gen_mule.py's own GPIO_PHYSICAL_PIN (imported, not
  duplicated, so the two can't silently drift apart) and to handle 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
Parts:
- removed D1, D10, D11, D12, D13, D14, D15, D16, D17, D2, D3, D4, D5, D6, D7, D8, D9: BAV99, symbol Diode:BAV99
- removed U5: PC847, symbol Isolator:PC847
- removed U6: TMA-0505S, symbol Converter_DCDC_Isolated:TMA-0505S
- removed U7: LD1117S33TR, symbol Regulator_Linear:AP1117-15
- added D1, D10, D11, D12, D13, D14, D15, D16, D17, D2, D3, D4, D5, D6, D7, D8, D9: BAT54S, symbol Diode:BAT54S
- added R26: 330, symbol Device:R
- added R27: 1k, symbol Device:R
- added U5, U6: HCPL-4661, symbol Isolator:HCPL-263A
- added U7: TMA-0505S, symbol Converter_DCDC_Isolated:TMA-0505S
- added U8: LD1117S33TR, symbol Regulator_Linear:AP1117-15
- R18: value 330 -> 100
- R19: value 4k7 -> 100
- R2, R4: value 100 -> 330
- R21, R23, R25: value 4k7 -> 1k
Connections:
- net U7_LED1 is gone; now on net EVT_D15_CLAMP: R18.2
- net +3V3: now also D1.2 (K), D10.2 (K), D11.2 (K), D12.2 (K), D13.2 (K), D14.2 (K), D15.2 (K), D16.2 (K), D17.2 (K), D2.2 (K), D3.2 (K), D4.2 (K), D5.2 (K), D6.2 (K), D7.2 (K), D8.2 (K), D9.2 (K), U8.2 (VO)
- net +5V: now also U7.1 (+Vin), U8.3 (VI)
- net BARCODE_ISO: now also R23.2, U5.6 (VO2); no longer R21.2
- net BARCODE_OUT: now also R22.1; no longer R20.1
- net BARCODE_PI: now also J2.11 (Pin_11); no longer J2.18 (Pin_18)
- net DGND: now also J2.6 (Pin_6), J2.9 (Pin_9), D1.1 (A), D10.1 (A), D11.1 (A), D12.1 (A), D13.1 (A), D14.1 (A), D15.1 (A), D16.1 (A), D17.1 (A), D2.1 (A), D3.1 (A), D4.1 (A), D5.1 (A), D6.1 (A), D7.1 (A), D8.1 (A), D9.1 (A), U5.2 (C1), U5.3 (C2), U6.2 (C1), U6.3 (C2), U7.2 (-Vin), U8.1 (GND); no longer J2.19 (Pin_19), J2.20 (Pin_20)
- net EVT_D0_CLAMP: now also D1.3 (COM)
- net EVT_D0_PI: now also J2.27 (Pin_27), R2.2; no longer J2.1 (Pin_1), U1.18 (Y0)
- net EVT_D10_CLAMP: now also R13.2, D11.3 (COM); no longer R11.2
- net EVT_D10_PI: now also J2.19 (Pin_19); no longer J2.11 (Pin_11)
- net EVT_D10_TPC: now also R13.1; no longer R11.1
- net EVT_D11_CLAMP: now also R14.2, D12.3 (COM); no longer R12.2
- net EVT_D11_PI: now also J2.23 (Pin_23); no longer J2.12 (Pin_12)
- net EVT_D11_TPC: now also R14.1; no longer R12.1
- net EVT_D12_CLAMP: now also R15.2, D13.3 (COM); no longer R13.2
- net EVT_D12_PI: now also J2.32 (Pin_32); no longer J2.13 (Pin_13)
- net EVT_D12_TPC: now also R15.1; no longer R13.1
- net EVT_D13_CLAMP: now also R16.2, D14.3 (COM); no longer R14.2
- net EVT_D13_PI: now also J2.33 (Pin_33); no longer J2.14 (Pin_14)
- net EVT_D13_TPC: now also R16.1; no longer R14.1
- net EVT_D14_CLAMP: now also R17.2, D15.3 (COM); no longer R15.2
- net EVT_D14_PI: now also J2.8 (Pin_8); no longer J2.15 (Pin_15)
- net EVT_D14_TPC: now also R17.1; no longer R15.1
- net EVT_D15_CLAMP: now also D16.3 (COM); no longer R16.2
- net EVT_D15_PI: now also J2.10 (Pin_10); no longer J2.16 (Pin_16)
- net EVT_D15_TPC: now also R18.1; no longer R16.1
- net EVT_D1_CLAMP: now also R3.2, D2.3 (COM); no longer R2.2
- net EVT_D1_PI: now also J2.28 (Pin_28), R4.2; no longer J2.2 (Pin_2), U1.17 (Y1)
- net EVT_D1_TPC: now also R3.1; no longer R2.1
- net EVT_D2_CLAMP: now also R5.2, D3.3 (COM); no longer R3.2
- net EVT_D2_TPC: now also R5.1; no longer R3.1
- net EVT_D3_CLAMP: now also R6.2, D4.3 (COM); no longer R4.2
- net EVT_D3_PI: now also J2.5 (Pin_5); no longer J2.4 (Pin_4)
- net EVT_D3_TPC: now also R6.1; no longer R4.1
- net EVT_D4_CLAMP: now also R7.2, D5.3 (COM); no longer R5.2
- net EVT_D4_PI: now also J2.7 (Pin_7); no longer J2.5 (Pin_5)
- net EVT_D4_TPC: now also R7.1; no longer R5.1
- net EVT_D5_CLAMP: now also R8.2, D6.3 (COM); no longer R6.2
- net EVT_D5_PI: now also J2.29 (Pin_29); no longer J2.6 (Pin_6)
- net EVT_D5_TPC: now also R8.1; no longer R6.1
- net EVT_D6_CLAMP: now also R9.2, D7.3 (COM); no longer R7.2
- net EVT_D6_PI: now also J2.31 (Pin_31); no longer J2.7 (Pin_7)
- net EVT_D6_TPC: now also R9.1; no longer R7.1
- net EVT_D7_CLAMP: now also R10.2, D8.3 (COM); no longer R8.2
- net EVT_D7_PI: now also J2.26 (Pin_26); no longer J2.8 (Pin_8)
- net EVT_D7_TPC: now also R10.1; no longer R8.1
- net EVT_D8_CLAMP: now also R11.2, D9.3 (COM); no longer R9.2
- net EVT_D8_PI: now also J2.24 (Pin_24); no longer J2.9 (Pin_9)
- net EVT_D8_TPC: now also R11.1; no longer R9.1
- net EVT_D9_CLAMP: now also R12.2, D10.3 (COM); no longer R10.2
- net EVT_D9_PI: now also J2.21 (Pin_21); no longer J2.10 (Pin_10)
- net EVT_D9_TPC: now also R12.1; no longer R10.1
- net EVT_STROBE_CLAMP: now also R19.2, D17.3 (COM); no longer R17.2
- net EVT_STROBE_ISO: now also R21.2, U5.7 (VO1); no longer R19.2
- net EVT_STROBE_PI: now also J2.36 (Pin_36), R20.1; no longer J2.17 (Pin_17), R18.1
- net EVT_STROBE_TPC: now also R19.1; no longer R17.1
- net ISO_5V: now also R27.1, U5.8 (VCC), U6.8 (VCC), U7.6 (+Vout); no longer R19.1
- net ISO_GND: now also U5.5 (GND), U6.5 (GND), U7.4 (-Vout)
- net OPTO_SPARE1_IN: now also R24.1; no longer R22.1
- net OPTO_SPARE1_ISO: now also R25.2, U6.7 (VO1); no longer R23.2
- net OPTO_SPARE2_IN: now also R26.1; no longer R24.1
- net OPTO_SPARE2_ISO: now also R27.2, U6.6 (VO2); no longer R25.2
- net U7_LED2 renamed U5_LED1
- net U5_LED1: now also U5.1 (A1)
- net U7_LED3 renamed U5_LED2
- net U5_LED2: now also U5.4 (A2)
- net U7_LED4 renamed U6_LED1
- net U6_LED1: now also U6.1 (A1)
- new net EVT_D0_BUF: R2.1, U1.18 (Y0)
- new net EVT_D1_BUF: R4.1, U1.17 (Y1)
- new net U6_LED2: R26.2, U6.4 (A2)
Other:
- note added: "GPIO0/GPIO1 -- physical pins 27/28 -- are probed by the Pi as I2C at boot,"
- note added: "looking for a HAT ID EEPROM. The 330R series resistors above limit contention"
- note added: "with that probe. Requires force_eeprom_read=0 in config.txt."

Commit message: fix(hw): clamp high side to +5V, not +3V3 -- coordinator caught own error
Fix round 2: the coordinator's own fix round 1 instruction to clamp the
inbound lines' high side to +3V3 was electrically wrong, and the
concern flagged in that round's report turned out to be the actual
bug, not a minor residual. SN74LVC541A is chosen specifically because
its inputs tolerate 5.5V independent of its own 3.3V supply -- a clamp
diode to +3V3 defeats exactly that property, permanently, since the
task PC's normal 5V logic-high sits ~1.7V above +3V3+Vf. That is not a
fault-only clamp, it is a continuous conduction path (~13.5mA/line,
~230mA worst case across 17 lines) into a 3.3V rail with no way to
sink it, present on every code the task PC emits.

bidirectional_clamp() in hardware/gen/gen_mule.py now references +5V
instead of +3V3 for the high-side clamp target. BAT54S stays the part,
stays wired as the series pair it is (signal -> pin 3 COM, DGND ->
pin 1, now +5V -> pin 2). Sanity check (task-2-report.md): under a
normal 5V logic-high, signal and +5V are both nominally 5V, so the
high-side diode sees ~0V of forward bias -- well under a Schottky's
~0.35V threshold -- and conducts leakage current only, not milliamps.
+5V+Vf (~5.3-5.4V) still sits comfortably under the LVC541A's 6.5V
absolute-maximum input rating, so a genuine overvoltage fault is still
caught.

hardware/gen/check_mule_netlist.py gained a new assertion: every one
of the 17 clamp diodes has exactly one pin on +5V, zero pins on +3V3,
and exactly one pin on DGND -- checked per-diode so a future edit
reintroducing +3V3 on even one of the 17 is caught, not just "is +5V
mentioned somewhere". Negative-control tested (moving one diode back
to +3V3 in a parsed copy and confirming verify() raises) before
committing.

ERC: 0 errors, 0 warnings. Direct netlist inspection confirms +3V3's
net membership no longer includes any diode reference at all, and all
17 diode references now appear on +5V.

Co-Authored-By: Claude Opus 5 (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
Connections:
- net +3V3: no longer D1.2 (K), D10.2 (K), D11.2 (K), D12.2 (K), D13.2 (K), D14.2 (K), D15.2 (K), D16.2 (K), D17.2 (K), D2.2 (K), D3.2 (K), D4.2 (K), D5.2 (K), D6.2 (K), D7.2 (K), D8.2 (K), D9.2 (K)
- net +5V: now also D1.2 (K), D10.2 (K), D11.2 (K), D12.2 (K), D13.2 (K), D14.2 (K), D15.2 (K), D16.2 (K), D17.2 (K), D2.2 (K), D3.2 (K), D4.2 (K), D5.2 (K), D6.2 (K), D7.2 (K), D8.2 (K), D9.2 (K)

Commit message: fix(hw): opto bypass caps, matched LED drive, all-8 grounds, permutation-proof checker
Fix round 3: task review came back spec-fail with one critical and four
important findings, all real.

CRITICAL -- no 0.1uF bypass on U5/U6 (HCPL-4661) or U7 (TMA-0505S).
Brief Step 4 asked for 100nF per IC; only U1-U4 got one. Added 100nF
between VCC/GND on both HCPL-4661 packages (within ~7mm per its
datasheet, noted for Task 3 layout), and on both the input and output
sides of the isolated DC-DC. Without it, an open-collector logic
optocoupler is prone to output chatter on transitions -- directly
compromising the propagation-delay/edge-quality measurement this board
exists to take (bring-up checks 5-6), which Task 11 reuses verbatim.

IMPORTANT 1 -- asymmetric opto LED drive. 330R on all four channels
gave ~4.8mA on the 3.3V-driven strobe channel against ~10mA on the
5V-driven barcode channel -- strobe sat below HCPL-4661's ~6.3mA
minimum I_F(on), and this family's propagation delay is strongly
I_F-dependent, so the two measured channels wouldn't transfer cleanly
to the real board. Strobe's resistor changed 330R -> 160R, landing
at exactly 10.0mA (barcode stays 330R/10.0mA) -- matched, not just
both above minimum. Spare (bench-injection) channels stay at 330R,
their drive voltage being unknown at generation time.

IMPORTANT 2 -- only 2 of the Pi header's 8 real ground pins were
bonded. The real board bonds all 8; a mule that bonds 2 doesn't
produce crosstalk/edge-quality measurements that transfer, which is
the board's whole purpose. PI_GND_PHYSICAL_PINS now lists all 8 real
positions (6, 9, 14, 20, 25, 30, 34, 39).

IMPORTANT 3 -- the netlist checker verified each net in isolation and
could not detect a channel permutation: nothing tied channel i's input
path to channel i's output path. hardware/gen/check_mule_netlist.py's
verify() now walks each of the 17 event-code channels end to end in
one function (_walk_channel): TPC header -> series R -> clamp node ->
buffer input pin -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
Parts:
- added C10, C11, C12: 10uF, symbol Device:C
- added C9: 100nF, symbol Device:C
- C6, C7, C8: value 10uF -> 100nF
- R20: value 330 -> 160
Connections:
- net +3V3: now also C11.1, C9.1; no longer C5.1, C7.1
- net +5V: now also C7.1, C10.1; no longer C6.1
- net DGND: now also J2.14 (Pin_14), J2.20 (Pin_20), J2.25 (Pin_25), J2.30 (Pin_30), J2.34 (Pin_34), J2.39 (Pin_39), C10.2, C11.2, C9.2; no longer C5.2, C6.2
- net ISO_5V: now also C5.1, C6.1, C12.1
- net ISO_GND: now also C5.2, C6.2, C12.2
- no-connect marks 55 -> 49

Commit message: feat(hw): mule layout, DRC clean, fab outputs
Adds hardware/gen/kicad_pcb.py (a .kicad_pcb generator mirroring kicad_sch.py's
technique: real footprints extracted from KiCad's stock .pretty libraries, placed
rigidly, nets assigned per pad straight from the schematic's own exported netlist)
and hardware/gen/gen_mule_pcb.py, which uses it to place all 72 mule components
per hardware/mule/floorplan.md: task-PC and Pi IDC-40 headers on opposite edges,
a single straight >=2.5mm isolation slot with the two HCPL-4661s and the isolated
DC-DC straddling it by design, everything else grouped by electrical domain either
side. `kicad-cli` has no netlist-import or Specctra-DSN subcommand, so there is no
headless path to routing -- this generates outline, placement and netlist import
only; a person routes it in pcbnew.

DRC: 0 courtyard/clearance/solder-mask errors. 210 unconnected-item errors (expected,
nothing is routed yet) and 10 warnings, all investigated in floorplan.md (8x
silk-vs-slot clearance on the 3 straddling parts, inherent to straddling by design;
2x a KiCad-internal lib_footprint_mismatch quirk specific to rotated instances,
confirmed independent of this generator's content via a standalone test).

Also closes out items Task 2's review deferred to this task:
- Footprints assigned from the real part being fitted (TSSOP-20, DIP-8, SOT-223,
  SOT-23, SIP-7), not the stand-in symbols' own filter suggestions -- gen_mule.py
  now passes a real footprint at every placement, which Sch.place() already
  supported but nothing used. Sch gained footprints/instance_uuid/values maps so
  the PCB generator has a single source of truth for role, footprint and value
  per reference instead of re-deriving them.
- Barrel-jack pin mapping re-confirmed against the actual datasheet of the jack
  whose footprint is now assigned (Same Sky/CUI PJ-102AH): matches Task 2's
  symbol-geometry inference exactly (pin 1 sleeve/DGND, pin 2 tip/+5V).
- Back-powering-through-the-clamps note carried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
Parts:
- C1, C2, C3, C4, C5, C6, C7, C8, C9: footprint (none) -> Capacitor_SMD:C_0603_1608Metric
- C10, C11, C12: footprint (none) -> Capacitor_SMD:C_0805_2012Metric
- D1, D10, D11, D12, D13, D14, D15, D16, D17, D2, D3, D4, D5, D6, D7, D8, D9: footprint (none) -> Package_TO_SOT_SMD:SOT-23
- J1, J2: footprint (none) -> Connector_PinHeader_2.54mm:PinHeader_2x20_P2.54mm_Vertical
- J3: footprint (none) -> Connector_PinHeader_2.54mm:PinHeader_1x04_P2.54mm_Vertical
- J4: footprint (none) -> TerminalBlock_Phoenix:TerminalBlock_Phoenix_MKDS-1,5-4_1x04_P5.00mm_Horizontal
- J5, J6, J7: footprint (none) -> Connector_PinHeader_2.54mm:PinHeader_1x02_P2.54mm_Vertical
- J8: footprint (none) -> Connector_BarrelJack:BarrelJack_CUI_PJ-102AH_Horizontal
- R1, R10, R11, R12, R13, R14, R15, R16, R17, R18, R19, R2, R20, R21, R22, R23, R24, R25, R26, R27, R3, R4, R5, R6, R7, R8, R9: footprint (none) -> Resistor_SMD:R_0603_1608Metric
- U1, U2, U3, U4: footprint (none) -> Package_SO:Texas_PW0020A_TSSOP-20_4.4x6.5mm_P0.65mm
- U5, U6: footprint (none) -> Package_DIP:DIP-8_W7.62mm
- U7: footprint (none) -> Converter_DCDC:Converter_DCDC_TRACO_TMA-05xxS_12xxS_Single_THT
- U8: footprint (none) -> Package_TO_SOT_SMD:SOT-223-3_TabPin2
