File: hardware/mule/mule.kicad_pcb (KiCad board)
At the start: 2 copper layers, 100 x 90 mm, 72 parts, among them J1 IDC-40 task-PC event bus, J2 IDC-40 Pi event bus, J3 BARCODE_OUT test points, J4 Isolated-domain outputs, J5 Opto spare 1 bench injection, J6 Opto spare 2 bench injection, J7 ISO_5V/ISO_GND test point, J8 +5V DC in, U1 SN74LVC541APW, U2 SN74LVC541APW, U3 SN74LVC541APW, U4 SN74HCT541PW, U5 HCPL-4661, U6 HCPL-4661, U7 TMA-0505S, U8 LD1117S33TR

Commit message: fix(hw): opto bypass caps within 7mm on both legs, rotation-correct instances
gen_mule_pcb.py's placement comment put U5's GND pin (pad 5) at (27.62, 70.12);
at rot=270 it lands at (12.38, 70.12), mirrored about the package. Both bypass
caps were placed at the midpoint of the VCC pin and that wrong coordinate, so
the copper was wrong, not just the comment: measured out of the committed board
file, each cap sat 3.85mm from VCC and 12.43mm from GND, against the HCPL-4661
datasheet's ~7mm, on the one board built to measure this optocoupler's edges.

Fixed at the source. kicad_pcb.py now derives placed geometry from the library
footprint itself -- place_point()/local_point() (transform verified against
kicad-cli pcb drc's own reported pad coordinates), footprint_pads(),
footprint_courtyard(), Board.pad_pos(), Board.courtyard() -- plus
read_placed_pads(), which re-measures pad positions out of a written .kicad_pcb
independently of the arithmetic that produced it. gen_mule_pcb.py places each
cap from its optocoupler's placed geometry, matches cap pad to IC pin by net,
and asserts both legs at placement time and again after re-reading the file.
As built, read back from mule.kicad_pcb: all four legs 3.74mm.

Also fixes two real construction differences against how pcbnew writes a
rotated footprint, found by diffing against KiCad's own demo boards:

- A placed pad's or text element's (at X Y ANGLE) angle is absolute, so a
  rotated instance needs library angle + rotation on every pad and text child.
  This is what kicad-cli pcb drc was reporting as lib_footprint_mismatch, not a
  KiCad quirk as previously recorded: reverting only this change brings the two
  warnings back, reverting only the point fix does not. Silent here (every
  DIP-8 pad is a circle or a square roundrect) and a genuine geometry error for
  any oval, rectangular, keyed or chamfered pad -- the same footprint plotted
  at rot=90 both ways gives apertures O,1.6X2.4 against O,2.4X1.6.
- A placed `point` (pin-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
Parts:
- moved C5 7.61 mm to (16.2, 72.3), turned to 180 degrees
- moved C6 7.61 mm to (40.2, 72.3), turned to 180 degrees
