File: hardware/breakout/sheets/taskpc-digital.kicad_sch (KiCad schematic)
At the start: 63 parts, among them J2 Connector 0 (analog + AISENSE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, J3 Connector 1 (digital, task PC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, J4 Manual reward button (panel), J5 Remote reward jack (parallel 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, J6 Reward driver out (BNC, place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, U10 SN74AHCT541PW, U11 SN74AHCT541PW, U12 SN74HCT32D, U13 SN74HCT14D, U5 SN74LVC541APW, U6 SN74LVC541APW, U7 SN74LVC541APW, U8 SN74AHCT541PW, U9 SN74AHCT541PW

Commit message: feat(breakout): manual reward one-shot and real BNC/pushbutton reward connectors
Change A: insert a Nexperia 74HCT123D monostable (U69) between the debounce
inverter and the reward-OR gate so every hand-delivered reward gets a fixed
~199ms pulse regardless of hold time (442k Rext / 1uF Cext, K=0.45 at 5V,
cross-checked against the datasheet's own measured example). Debounce RC
changes from 10k x 100nF to 10k x 1uF (~10ms), covering switch bounce and
the longer remote-BNC cable run's own mating transient. Pin map verified
against Nexperia's real datasheet (TI's own CD74HCT123M/MT is obsolete).

Change B: the three reward panel positions become real connectors -- J4
(button) is a recessed panel pushbutton (Button_Switch_THT:SW_PUSH-12mm),
J5/J6 are real BNCs, replacing generic Conn_01x02 placeholders. This removes
the 3.5mm TRS from the design entirely (no TRS footprint/symbol exists
anywhere on the board, confirmed by grep and by a whole-board checker scan).
J4/J5/J6 keep their existing reference numbers.

Also fixes a real ref_start staleness hazard found while implementing this:
taskpc-digital.kicad_sch's own build() re-derived its reference-counter seed
from power.kicad_sch's *current* text on every regeneration, which silently
renumbers this sheet's own existing components once an earlier sibling
sheet (power.kicad_sch, via its fan-header addendum) has drifted since this
sheet was last generated. Fixed by pinning ref_start to the historically
correct values; the identical fix lands on pi-interface.kicad_sch's own
build() for the same reason.

Extended check_taskpc_digital_netlist.py with the one-shot topology walk,
reward-connector footprint checks, and a whole-board "no 3.5mm TRS anywhere"
scan, each with a genuinely-firing negative control. Also wires in the
shared row-pitch collision guard (not previously used by this checker) --
it caught this task's own initial row-spacing mistake, since fixed.

kicad-cli sch erc: 0 errors, 3 pre-existing warnings (unchanged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
Parts:
- removed J4: Manual reward button (panel), Connector_PinHeader_2.54mm:PinHeader_1x02_P2.54mm_Vertical, symbol Connector_Generic:Conn_01x02
- removed J5: Remote reward jack (parallel to panel button), Connector_PinHeader_2.54mm:PinHeader_1x02_P2.54mm_Vertical, symbol Connector_Generic:Conn_01x02
- removed J6: Reward driver out (BNC, placeholder), Connector_PinHeader_2.54mm:PinHeader_1x02_P2.54mm_Vertical, symbol Connector_Generic:Conn_01x02
- added C149: 1uF, Capacitor_SMD:C_0603_1608Metric, symbol Device:C
- added C150: 100nF, Capacitor_SMD:C_0603_1608Metric, symbol Device:C
- added J4: Manual reward button (panel, recessed), Button_Switch_THT:SW_PUSH-12mm, symbol Switch:SW_Push
- added J5: Remote reward BNC (parallel to panel button; lock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, Connector_Coaxial:BNC_PanelMountable_Vertical, symbol Connector:Conn_Coaxial
- added J6: Reward driver out (BNC), Connector_Coaxial:BNC_PanelMountable_Vertical, symbol Connector:Conn_Coaxial
- added R191: 442k, Resistor_SMD:R_0603_1608Metric, symbol Device:R
- added U69: 74HCT123D, Package_SO:SOIC-16_3.9x9.9mm_P1.27mm, symbol 74xx:74HCT123
- C29: value 100nF -> 1uF
Connections:
- net +5V: now also C150.1, R191.1, U69.16 (VCC), U69.3 (Clr)
- net DGND: now also C150.2, J4.2, J5.2 (Ext), J6.2 (Ext), U69.1 (A), U69.10 (B), U69.11 (Clr), U69.6 (Cext), U69.7 (RCext), U69.8 (GND), U69.9 (A)
- net RWD_BTN: now also J4.1, J5.1 (In)
- net RWD_BTN_DEB: now also U69.2 (B); no longer U12.2
- net RWD_DLVR: now also J6.1 (In)
- new net RWD_BTN_PULSE: U12.2, U69.13 (Q)
- new net U69_CEXT: C149.2, U69.14 (Cext)
- new net U69_RCEXT: C149.1, R191.2, U69.15 (RCext)
- no-connect marks 106 -> 109
Other:
- note added: "'how long the button is held'."
- note added: "(10k pull-up to +5V), reads LOW while pressed. A SINGLE 74HCT14 Schmitt"
- note added: "(datasheet Table 10, HCT-specific) = 0.45 x 442 x 1e6 = 198.9e6 ns = ~199ms."
- note added: "(idle-LOW, pulses HIGH on delivery -- this design's other event lines' own"
- note added: "+5V -> R191(442k) -> pin15(REXT/CEXT) -> C149(1uF) -> pin14(CEXT) -- R and C"
- note added: "A=DGND, B=RWD_BTN_DEB (trigger, rising edge), RD-bar=+5V (never reset) --"
- note added: "ALREADY-DEBOUNCED RWD_BTN_DEB (bounce filtered upstream), so hold duration"
- note added: "Cross-checked against the SAME table's own measured example (Cext=100nF,"
- note added: "HIGH polarity, unchanged requirement. RWD_CMD polarity is ASSUMED ACTIVE-HIGH"
- note added: "MANUAL REWARD ONE-SHOT (panel-instrumentation task, 2026-08-15, spec Sec.3.1):"
- note added: "Nexperia 74HCT123D (TI's own CD74HCT123M/MT is obsolete, checked before"
- note added: "Retriggerable by design (datasheet Section 1) -- deliberately not worked"
- note added: "Reward OR polarity (fix round 1, finding 1 -- CRITICAL): RWD_BTN idles HIGH"
- note added: "RewardPolarity setting must be HIGH to match this board -- hardware/README.md):"
- note added: "Rext=10k -> Typ=450us; formula predicts 450us exactly)."
- note added: "Rext=442k (E96), Cext=1uF: tW = K x Rext[kOhm] x Cext[pF], K=0.45 at VCC=5.0V"
- note added: "Second section (unit 2) held in PERMANENT RESET (RD-bar->DGND, datasheet"
- note added: "Table 4 row 1) -- genuinely inert, not merely untriggered. Pin map verified"
- note added: "U69 (Nexperia 74HCT123D) gives every hand-delivered reward a FIXED ~199ms"
- note added: "actual polarity against MonkeyLogic before commissioning (MonkeyLogic's own"
- note added: "an OR gate cannot correctly combine one active-HIGH and one active-LOW input."
- note added: "around: a single continuous hold produces exactly one rising edge on the"
- note added: "cannot extend the pulse; retriggering only matters for a second physical"
- note added: "checked against KiCad's own 74xx:74HCT123 library entry -- see"
- note added: "choosing this vendor, not assumed from the symbol's own generic library name)."
- note added: "commanded (RWD_CMD) and delivered (RWD_DLVR) separately at all: a manual"
- note added: "convention, and SN74LVC541APW does not invert): stated explicitly because this"
- note added: "countable, not a per-press variable, which is the point of recording"
- note added: "datasheet Table 4's own function table, row 'nRD=H,nA=L,nB=up-arrow', fires"
- note added: "in series sharing one node, per TI SLVA720A Fig.3-1's own topology, NOT each"
- note added: "independently returned to a rail."
- note added: "inverter (NOT a pair) inverts ONCE, so RWD_BTN_DEB idles LOW and reads HIGH"
- note added: "one pulse on B's own rising edge. Q=RWD_BTN_PULSE (active-HIGH). RC network:"
- note added: "output, RWD_BTN_PULSE, is what actually reaches the OR gate -- same active-"
- note added: "pin-by-pin against Philips/Nexperia Rev.03 (11 May 2004) Table 3/Fig.5, cross-"
- note added: "place_reward_oneshot()'s own docstring for the full account. Real part:"
- note added: "press inside the first pulse's own ~199ms window, a different scenario than"
- note added: "pulse regardless of how long RWD_BTN is held -- so a manual reward is"
- note added: "reward is DELIVERED WITHOUT COMMANDED, derivable with no extra logic."
- note added: "sheet cannot verify the task PC/MonkeyLogic side independently. VERIFY RWD_CMD's"
- note added: "while pressed -- active-HIGH. RWD_BTN_DEB now feeds a one-shot (74HCT123D,"
- note added: "~199ms fixed pulse -- panel-instrumentation task, 2026-08-15) whose own Q"
- note removed: "74HCT14 Schmitt inverter (NOT a pair -- a pair was this task's own pre-fix-"
- note removed: "LOW input regardless of the button side's own inverter count."
- note removed: "MonkeyLogic before commissioning: if active-HIGH as assumed, this OR gate is"
- note removed: "MonkeyLogic side independently. VERIFY RWD_CMD's actual polarity against"
- note removed: "ORed with an active-HIGH RWD_CMD asserts RWD_DLVR permanently) inverts ONCE,"
- note removed: "RWD_BTN idles HIGH (10k pull-up to +5V), reads LOW while pressed. A SINGLE"
- note removed: "RWD_CMD polarity is ASSUMED ACTIVE-HIGH (idle-LOW, pulses HIGH on delivery --"
- note removed: "Reward OR polarity (fix round 1, finding 1 -- CRITICAL, corrected here):"
- note removed: "correct; an OR gate cannot correctly combine one active-HIGH and one active-"
- note removed: "invert): stated explicitly because this sheet cannot verify the task PC/"
- note removed: "round-1 defect: 2 series stages cancel, leaving RWD_BTN_DEB idle-HIGH, which"
- note removed: "so RWD_BTN_DEB idles LOW and reads HIGH while pressed -- active-HIGH."
- note removed: "this design's other event lines' own convention, and SN74LVC541APW does not"

Commit message: fix(hardware): drive the optocoupler LEDs (F1, both halves)
430R never switched these LEDs. The original sizing solved
(5.0 - V_OL - V_F)/I correctly but against the rail's NOMINAL 5.00V and
V_F TYP; +5V reaches the anodes through F4 and D3 (0.42-0.49V of drop)
and V_F's worst case is 1.80V, so the real worst-case current was ~5mA
against the ACSL-6xx0's 7.0mA I_FH minimum. 30 channels were not
guaranteed to switch for seventy-three commits.

Both halves land together because neither is shippable alone -- 430R
starves the LED, and 249R (~12.7mA) overloads a single 7.5mA output.

Resistors, rail-aware: 430R -> 249R on the 30 LEDs fed from +5V, ->
301R on the 2 fed from ISO_5V. ISO_5V is regulated locally with nothing
in series, so 249R there would give 15.1mA -- past the 15mA ABSOLUTE
maximum. One value is wrong on one rail or the other.

Paralleling: every buffer-driven LED now has two SN74AHCT541 outputs
from tied inputs. Four new packages (U70-U73) plus C151-C154, 5 buffer
packages to 9, 6 spare channels. Channel maps are mirrored from the
tables that built the first leg rather than re-listed, so the legs
cannot drift apart. Refdes minted out of band, above the board maximum:
8 refs added, 0 removed, 0 renumbered.

This also fixes a per-PACKAGE limit no per-pin check could see. The
AHCT541's GND absolute maximum is 75mA (SCLS269Q 4.1, not the 100mA
hardware/README.md claimed); U8/U9 drive eight LEDs each; the drive is
active-low and the event bus idles at 0x0000, so sixteen LEDs are lit
CONTINUOUSLY. At 249R unparalleled that is ~101mA through one ground
pin. Paralleled it is 55.6mA worst case.

RHS_STIM_OUT's LED moves to a new buffered leg (RHS_STIM_OUT_BUF, off
U11's last two spare channels). It was the one channel driven by an
ACSL-6420 output rather than a buffer -- a deliberate, checked exception
that was correct at 430R (8.61mA of a 13mA budget) and not correct at
249R (13.85mA with its pull-up). The exception did not change; the
number it had been checked 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
Parts:
- added C151, C152, C153, C154: 100nF, Capacitor_SMD:C_0603_1608Metric, symbol Device:C
- added U70, U71, U72, U73: SN74AHCT541PW, Package_SO:Texas_PW0020A_TSSOP-20_4.4x6.5mm_P0.65mm, symbol 74xx:74AHCT541
Connections:
- net +5V: now also C151.1, C152.1, C153.1, C154.1, U70.20 (VCC), U71.20 (VCC), U72.20 (VCC), U73.20 (VCC)
- net DGND: now also C151.2, C152.2, C153.2, C154.2, U70.1 (G1), U70.10 (GND), U70.19 (G2), U71.1 (G1), U71.10 (GND), U71.19 (G2), U72.1 (G1), U72.10 (GND), U72.19 (G2), U73.1 (G1), U73.10 (GND), U73.19 (G2), U73.4 (A2), U73.5 (A3), U73.6 (A4), U73.7 (A5), U73.8 (A6), U73.9 (A7); no longer U11.8 (A6), U11.9 (A7)
- net EVT_D0_BUF: now also U70.18 (Y0)
- net EVT_D0_CLAMP: now also U70.2 (A0)
- net EVT_D10_BUF: now also U71.16 (Y2)
- net EVT_D10_CLAMP: now also U71.4 (A2)
- net EVT_D11_BUF: now also U71.15 (Y3)
- net EVT_D11_CLAMP: now also U71.5 (A3)
- net EVT_D12_BUF: now also U71.14 (Y4)
- net EVT_D12_CLAMP: now also U71.6 (A4)
- net EVT_D13_BUF: now also U71.13 (Y5)
- net EVT_D13_CLAMP: now also U71.7 (A5)
- net EVT_D14_BUF: now also U71.12 (Y6)
- net EVT_D14_CLAMP: now also U71.8 (A6)
- net EVT_D15_BUF: now also U71.11 (Y7)
- net EVT_D15_CLAMP: now also U71.9 (A7)
- net EVT_D1_BUF: now also U70.17 (Y1)
- net EVT_D1_CLAMP: now also U70.3 (A1)
- net EVT_D2_BUF: now also U70.16 (Y2)
- net EVT_D2_CLAMP: now also U70.4 (A2)
- net EVT_D3_BUF: now also U70.15 (Y3)
- net EVT_D3_CLAMP: now also U70.5 (A3)
- net EVT_D4_BUF: now also U70.14 (Y4)
- net EVT_D4_CLAMP: now also U70.6 (A4)
- net EVT_D5_BUF: now also U70.13 (Y5)
- net EVT_D5_CLAMP: now also U70.7 (A5)
- net EVT_D6_BUF: now also U70.12 (Y6)
- net EVT_D6_CLAMP: now also U70.8 (A6)
- net EVT_D7_BUF: now also U70.11 (Y7)
- net EVT_D7_CLAMP: now also U70.9 (A7)
- net EVT_D8_BUF: now also U71.18 (Y0)
- net EVT_D8_CLAMP: now also U71.2 (A0)
- net EVT_D9_BUF: now also U71.17 (Y1)
- net EVT_D9_CLAMP: now also U71.3 (A1)
- net EVT_STROBE_BUF: now also U72.18 (Y0)
- net EVT_STROBE_CLAMP: now also U72.2 (A0), U72.5 (A3)
- net EVT_STROBE_INTAN_BUF: now also U72.15 (Y3)
- net PD1_COMP: now also U73.2 (A0)
- net PD1_COMP_BUF: now also U73.18 (Y0)
- net PD2_COMP: now also U73.3 (A1)
- net PD2_COMP_BUF: now also U73.17 (Y1)
- net RHS_STIM_OUT: now also U11.8 (A6), U11.9 (A7)
- net RWD_CMD_BUF: now also U72.17 (Y1)
- net RWD_CMD_CLAMP: now also U72.3 (A1), U72.6 (A4)
- net RWD_CMD_INTAN_BUF: now also U72.14 (Y4)
- net RWD_DLVR: now also U72.8 (A6), U72.9 (A7)
- net RWD_DLVR_BUF: now also U72.12 (Y6)
- net RWD_DLVR_INTAN_BUF: now also U72.11 (Y7)
- net STIM_TRIG_BUF: now also U72.16 (Y2)
- net STIM_TRIG_CLAMP: now also U72.4 (A2), U72.7 (A5)
- net STIM_TRIG_INTAN_BUF: now also U72.13 (Y5)
- net RHS_STIM_OUT_BUF: now reaches U11.11 (Y7)
- net RHS_STIM_OUT_BUF: now also U11.12 (Y6)
- no-connect marks 109 -> 113
Other:
- note added: "(6 spare channels, the headroom finding F4's camera triggers need)"
- note added: "CONTINUOUSLY. At 249R unparalleled that is ~101mA through one ground pin."
- note added: "Each ACSL-6400/6420 LED on this board is fed from +5V through 249R and draws"
- note added: "Each pair shares ONE input net, and that is a safety requirement rather than"
- note added: "It also fixes a PACKAGE limit no per-pin check can see. AHCT541's GND-pin"
- note added: "LEDs were never guaranteed to switch (~5mA worst case against a 7.0mA I_FH"
- note added: "Paralleled it is ~51mA, and each output pin sees ~6.3mA of a 7.5mA budget."
- note added: "REFDES U70-U73/C151-C154 are minted OUT OF BAND (explicit strings, never"
- note added: "TWO BUFFER OUTPUTS PER OPTOCOUPLER LED (finding F1b, 2026-08-16)."
- note added: "The value cannot simply be reduced: it is pinned between the part's 7-15mA"
- note added: "These four packages carry the SECOND output of every LED pair. They exist"
- note added: "U69/R191/C149-C150 already use here. An ordinary next_ref() would renumber"
- note added: "U70 doubles U8 -- EVT_D0_BUF .. EVT_D7_BUF"
- note added: "U71 doubles U9 -- EVT_D8_BUF .. EVT_D15_BUF"
- note added: "U72 doubles U10 -- strobe/RWD_CMD/STIM_TRIG _BUF + the 5 second legs"
- note added: "U73 doubles U11's two LED channels -- PD1_COMP_BUF, PD2_COMP_BUF"
- note added: "absolute maximum is 75mA; U8 and U9 drive eight LEDs each; the drive is"
- note added: "active-low and the event bus idles at 0x0000, so sixteen LEDs are lit"
- note added: "because the LED series resistor had to fall from 430R to 249R -- at 430R the"
- note added: "every part placed after it AND every downstream sibling sheet."
- note added: "first leg rather than retyped, so the two cannot drift apart."
- note added: "guaranteed to drive the same direction. If their inputs ever differed, one"
- note added: "minimum, because the +5V rail reaches them through F4 and D3 and the original"
- note added: "next_ref()), above the whole board's current maximum -- the same mechanism"
- note added: "recommended band and its 7.0mA worst-case switching threshold. A driver pin"
- note added: "separately gives each SINGLE LED two outputs, which is the opposite thing."
- note added: "sizing used a nominal 5.00V and a TYPICAL V_F) -- and 249R draws ~12.7mA,"
- note added: "stages. The channel maps here are MIRRORED from the tables that built the"
- note added: "tidiness: two tri-state outputs on one net are safe only while both are"
- note added: "which one AHCT541 output cannot sink. Neither value is shippable alone."
- note added: "with TWO LEDs on it sinks double, which is what this note block is about; F1"
- note added: "would source while the other sinks, limited by nothing but the two output"
- note added: "written, which under-drove every LED on the board -- see the F1 note block)."
- note added: "~12.7mA as of finding F1 (2026-08-16; it was 430R/~7.33mA when this note was"
- note removed: "Each ACSL-6400/6420 LED on this board is fed from +5V through 430R and draws"
- note removed: "inside the part's 7-15mA recommended band and clear of its 7.0mA worst-case"
- note removed: "switching threshold, so it cannot simply be reduced). A driver pin with TWO of"
- note removed: "them sinks 14.7mA."
- note removed: "~7.33mA (gen_breakout_opto_ni.py's own derivation: the value is chosen to sit"
