File: hardware/breakout/sheets/taskpc-digital.kicad_sch (KiCad schematic)
At the start: 76 parts, among them J2 Connector 0 (analog + AISENSE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, J3 Connector 1 (digital, task PC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, J4 Manual reward button (panel, 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, J5 Dual panel BNC: Remote reward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, J6 Dual panel BNC: Reward driver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, U10 SN74AHCT541PW, U11 SN74AHCT541PW, U12 SN74HCT32D, U13 SN74HCT14D, U5 SN74LVC541APW, U6 SN74LVC541APW, U69 74HCT123D, U7 SN74LVC541APW, U70 SN74AHCT541PW, U71 SN74AHCT541PW, U72 SN74AHCT541PW, U73 SN74AHCT541PW, U8 SN74AHCT541PW, U9 SN74AHCT541PW

Commit message: Breakout: draw the task-PC line-out and the PFI copy of PD1_COMP
Implements hardware/breakout/line-out-and-pfi-copy.md (spec Sec.12 item 11,
wl-xcon XC-327), approved 2026-10-18.

- Line-out. Connector 0's AO 0/AO 1 (pins 22/21) go through R221/R222
  (100 ohm) to J57, a new isolated dual BNC on the back face. Its shells are on
  AO_GND_TPC (pins 55/54) and nothing else: NI ties AO GND to D GND on the card,
  so no board plane may carry the amplifier's return.
- PFI copy. pi-interface's SN74LVC541A level shifter gains channel 1, PD1_COMP ->
  PD1_COMP_PFI_BUF, which R223 (100 ohm) takes to Connector 0 pin 38, PFI 7.
  That pin avoids the default counter outputs, PFI 12-15. The departure from
  spec Sec.7.1's direction table is stated where it is made.
- D3 was reversed while drawing. Tying Connector 0's D GND to DGND made it a
  second component on both grounds after the star-point net tie, because its
  AISENSE is on AGND. check_breakout_power_netlist.py caught it. Pin 36 stays
  no-connect, and the checker now asserts that.

New refdes are out of band (J57, R221-R223, above the J56/R220 maxima). Only the
two changed sheets were regenerated, and no existing refdes moved on either.

Checks:
- both sheet checkers gained exact node assertions plus four mutations
  (shell on DGND, L/R swapped, copy on PFI 8, copy fed from a tied-off input);
- all ten checkers pass with their self-tests;
- ERC is unchanged (0 errors, the same 3 warnings);
- the netlist export reports no annotation errors;
- the netlist contract and both BOMs are updated, with the BOM count guards
  bumped deliberately.

Also corrects the generator's claim that P2 is on Connector 1. Panel
elevations: the back face goes to 10 bodies with 7.2 mm of slack, so nothing
more fits there. The wl-xcon reply names PFI 7 and the never-an-output rule.

Co-Authored-By: Claude Opus 5.5 (1M context) <noreply@anthropic.com>
Claude-Session: https://claude.ai/code/session_013HK81J55qfjevPUUfGjAqJ
Parts:
- added J57: Dual panel BNC: Line-out L (task PC AO 0) | Line-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, wl-sync:BNC_Dual_RA_Isolated, symbol wl-sync:BNC_Dual_RA_Isolated
- added R221, R222, R223: 100, Resistor_SMD:R_0603_1608Metric, symbol Device:R
Connections:
- net AO_R_TPC: now reaches J2.21
- net AO_R_TPC: now also R222.1
- net AO_L_TPC: now reaches J2.22
- net AO_L_TPC: now also R221.1
- net PD1_COMP_PFI: now reaches J2.38
- net PD1_COMP_PFI: now also R223.2
- net AO_GND_TPC: now reaches J2.54
- net AO_GND_TPC: now also J2.55, J57.2 (A_Ext), J57.4 (B_Ext)
- new net AO_L_BNC: J57.1 (A_In), R221.2
- new net AO_R_BNC: J57.3 (B_In), R222.2
- new net PD1_COMP_PFI_BUF: R223.1
- no-connect marks 114 -> 109
Other:
- note added: "AO GND=pins55,54=AO_GND_TPC (own net, no board plane) PFI7=pin38=PD1_COMP_PFI"
- note added: "Connector 1 = AI16-31 + P0.8-31, NO PFI (digital). See spec Sec.9.2, closed"
- note added: "Line-out and PFI copy (2026-10-18): AO0=pin22=AO_L_TPC AO1=pin21=AO_R_TPC"
- note added: "NI ties AO GND to D GND on the card, so no board plane may carry the amplifier's"
- note added: "No D GND pin here: AISENSE is already on AGND, and one connector on both grounds"
- note added: "Remaining 53 pins (spare AI9-15, P0.0-7, other PFI, D GND, +5V, NC) stay"
- note added: "Task-PC line-out and PD1_COMP's PFI copy (2026-10-18) -- see"
- note added: "breaks the single star point. All 16 PFI lines are on THIS connector (NI A-5)."
- note added: "hardware/breakout/line-out-and-pfi-copy.md. J57's shells are on AO_GND_TPC ONLY:"
- note added: "no_connect -- see _place_connector0()'s own docstring."
- note added: "out against the card's 2.2 V V_IH); PFI 7, not PFI 12-15, the default counter"
- note added: "outputs. Place R221-R223 beside Connector 0 in layout. Refdes out of band."
- note added: "return. PD1_COMP_PFI_BUF comes from pi-interface's SN74LVC541A channel 1 (3.3 V"
- note removed: "Connector 1 = AI16-31 + P0.8-31 + P2.0-7 (digital). See spec Sec.9.2, closed"
- note removed: "Remaining 58 pins (spare AI9-15, P0.0-7/P1.0-7/P2.x, D GND, +5V, AO*, NC) stay"
- note removed: "docstring."
- note removed: "no_connect: outside this task's own contract -- see _place_connector0()'s own"
