File: hardware/breakout/sheets/power.kicad_sch (KiCad schematic)
At the start: 44 parts, among them J1 M12A_5, J52 Chassis fan 1, J53 Chassis fan 2, J54 Chassis fan 3, J55 Chassis fan 4, U1 LD1117S33TR_SOT223, U2 IH1215D, U3 TPS7A4901, U4 TPS7A3001

Commit message: feat(breakout): chassis earth stud, power-good LEDs, rail test points, main fusing
Change D: five things a rack instrument needs that this board lacked
(spec Sec.9.8), four landing on power.kicad_sch and one on
pi-interface.kicad_sch:

- Chassis earth stud (J56): an M3 mounting hole with a connected pad --
  the mounting point spec Sec.5.6's cage-to-rack bond can land on. Carries
  a new CHASSIS_GND net, joined to DGND at exactly one net tie (NT3),
  mirroring the fan return's own NT2 treatment.
- Power-good LED per rail (D40/D41/D42, +12V/-12V/+5V): a failed rail is
  otherwise invisible until the data is wrong. ~4.5mA each, negligible
  against any rail's own budget.
- Rail test points (TP1-TP7): one per voltage rail plus one on INTAN_GND --
  the isolated domain's own reference, without which ISO_P12/ISO_N12
  cannot actually be measured (INTAN_GND is galvanically separate from
  AGND/DGND).
- Main input fusing (F2/F3/F4, +-12V/+5V): the fans already had a
  polyfuse; the main rails did not. Same real part as the fan feed's own
  F1 (Littelfuse 1206L050/15YR). A higher-current Bourns MF-SM alternative
  was evaluated and rejected: its own datasheet advises against hand
  soldering, which would add a third accepted hand-solderability exception
  beyond the two this board already documents. +-12V's own real total draw
  is flagged for bench confirmation rather than presented as fully closed.
- Barcode heartbeat LED (D43, on pi-interface.kicad_sch): a third
  dedicated leg off the trigger buffer's own BARCODE_RAW input, so the
  visible "sync box alive" LED never loads the real barcode net.

Extended check_breakout_power_netlist.py and
check_breakout_pi_interface_netlist.py with topology checks for every new
item, each with a genuinely-firing negative control, and wired in the
shared row-pitch collision guard where it was missing.

Regenerated hardware/breakout/netlist-contract.json and both BOM CSVs
(raw + order, +14 rows) against this cumulative state; updated
pro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
Parts:
- added D40, D41, D42: LED, LED_SMD:LED_0603_1608Metric_Pad1.05x0.95mm_HandSolder, symbol Device:LED
- added F2, F3, F4: 1206L050/15YR, Fuse:Fuse_1206_3216Metric_Pad1.42x1.75mm_HandSolder, symbol Device:Polyfuse
- added J56: Chassis earth stud, MountingHole:MountingHole_3.2mm_M3_Pad, symbol Connector_Generic:Conn_01x01
- added NT3: NetTie_2, NetTie:NetTie-2_SMD_Pad2.0mm, symbol Device:NetTie_2
- added R192, R193: 2.2k, Resistor_SMD:R_0603_1608Metric, symbol Device:R
- added R194: 680, Resistor_SMD:R_0603_1608Metric, symbol Device:R
- added TP1: +12V, TestPoint:TestPoint_THTPad_2.0x2.0mm_Drill1.0mm, symbol Connector:TestPoint
- added TP2: -12V, TestPoint:TestPoint_THTPad_2.0x2.0mm_Drill1.0mm, symbol Connector:TestPoint
- added TP3: +5V, TestPoint:TestPoint_THTPad_2.0x2.0mm_Drill1.0mm, symbol Connector:TestPoint
- added TP4: +3V3, TestPoint:TestPoint_THTPad_2.0x2.0mm_Drill1.0mm, symbol Connector:TestPoint
- added TP5: ISO_P12, TestPoint:TestPoint_THTPad_2.0x2.0mm_Drill1.0mm, symbol Connector:TestPoint
- added TP6: ISO_N12, TestPoint:TestPoint_THTPad_2.0x2.0mm_Drill1.0mm, symbol Connector:TestPoint
- added TP7: INTAN_GND, TestPoint:TestPoint_THTPad_2.0x2.0mm_Drill1.0mm, symbol Connector:TestPoint
Connections:
- net +12V: now also R192.1, TP1.1
- net +3V3: now also TP4.1
- net +5V: now also R194.1, TP3.1
- net -12V: now also D41.1 (K), TP2.1
- net AGND: now also D40.1 (K), R193.1
- net DGND: now also D42.1 (K), NT3.2
- net INTAN_GND: now also TP7.1
- net ISO_N12: now also TP6.1
- net ISO_P12: now also TP5.1
- net N12_RAW: now also F3.1; no longer D2.1 (K)
- net P12_RAW: now also F2.1; no longer D1.2 (A)
- net P5_RAW: now also F4.1; no longer D3.2 (A)
- new net CHASSIS_GND: J56.1 (Pin_1), NT3.1
- new net N12_FUSED: D2.1 (K), F3.2
- new net P12_FUSED: D1.2 (A), F2.2
- new net P5_FUSED: D3.2 (A), F4.2
- new net PGOOD_D40: D40.2 (A), R192.2
- new net PGOOD_D41: D41.2 (A), R193.2
- new net PGOOD_D42: D42.2 (A), R194.2
Other:
- note added: "(INTAN_GND is galvanically separate from AGND/DGND, Sec.5.3/5.5)."
- note added: "(Item 5, barcode heartbeat LED, is not on this sheet -- it lives on"
- note added: "1. Chassis earth stud (J56): a mounting point the cage-to-rack bond (Sec.5.6)"
- note added: "1206L050/15YR) as F1, placed upstream of each rail's own existing"
- note added: "2. Power-good LED per rail (D40/D41/D42, +12V/-12V/+5V): a failed rail is"
- note added: "3. Rail test points (TP1-7): one per voltage rail (+12V/-12V/+5V/+3V3/"
- note added: "4. Main input fusing (F2/F3/F4, +12V/-12V/+5V): the fans already had a"
- note added: "AGND/DGND themselves are not dedicated here -- already trivially"
- note added: "FAN_RTN's own NT2 -- reaches the board's single star point transitively."
- note added: "ISO_P12/ISO_N12) PLUS one on INTAN_GND -- the isolated rails' own"
- note added: "PANEL-INSTRUMENTATION ADDITIONS (2026-08-15, spec Sec.9.8) -- five things a"
- note added: "against any rail's own real budget."
- note added: "buffer already placed there, per spec Sec.9.8's own instruction not to"
- note added: "can land on. CHASSIS_GND joins DGND at exactly one point (NT3), mirroring"
- note added: "docstring for the sizing and the +-12V margin caveat."
- note added: "load the barcode net itself.)"
- note added: "otherwise invisible until the data is wrong. ~4.5mA each, negligible"
- note added: "pi-interface.kicad_sch, driven from a spare buffered leg of the trigger"
- note added: "polyfuse (F1); the main rails did not. Same real part (Littelfuse"
- note added: "probable at any of this sheet's own many ground pads."
- note added: "rack instrument needs that this board lacked; all landing on this sheet:"
- note added: "reference, without which ISO_P12/ISO_N12 cannot be measured at all"
- note added: "reverse-polarity diode (_place_inlet()) -- see that function's own"

Commit message: fix(hardware): give the fan branch its own fuse path, and size F4 for the real +5V load (F7, M7)
F7 -- THE FAN FUSE WAS DEFEATED BY ITS OWN PLACEMENT.

F1 was fed from +12V, which is downstream of F2:

    J1.1 -> P12_RAW -> [F2] -> P12_FUSED -> [D1] -> +12V -> [F1] -> FAN_12V

so the two were in SERIES at identical ratings (0.5 A hold / 1.0 A trip).
Two identical parts in series have no selectivity: a fan fault at 0.9 A is
below F1's trip but well over F2's hold, so F2 can open first and kill the
analog rails to protect the fans -- inverting the whole purpose of giving
the fans a separate fuse. It also meant F2 carried 337-361 mA rather than
the ~100 mA the main rail alone draws.

The fan branch now taps P12_RAW, with its own reverse-polarity Schottky
(D44, SS14) since it no longer sits behind D1:

    J1.1 -> P12_RAW -+- [F2] -> P12_FUSED   -> [D1]  -> +12V
                     `- [F1] -> FAN_12V_RAW -> [D44] -> FAN_12V

NOT WHAT THE AUDIT'S OWN F7 FIX LINE SAYS. It names P12_FUSED and calls it
"upstream of F2", but P12_FUSED is F2's OUTPUT -- tapping there would have
left fan current flowing through F2 while stripping the fan branch of
reverse-polarity protection, which is strictly worse than the defect. The
handoff's preferred option (tap P12_RAW, add a diode) is correct and is
what shipped. Both documents now record the correction.

M7 -- F4 WOULD HAVE TRIPPED IN NORMAL OPERATION.

The +5 V rail carries 392 mA typ / 495 mA max once finding F1 raised the
optocoupler drive, and 1206L050 holds only ~0.44 A at this chassis's 35 C
ambient. F4 -> 1206L110-C (1.10 A hold / 2.20 A trip, ~0.97 A derated, a
1.97x margin).

The audit left open whether a 1.1 A PPTC exists in 1206 at all, and whether
the answer forced a third package exception (against a global limit of two)
or splitting +5 V into two fused branches. It exists, so neither is needed.
Its lower R_min (0.040 vs 0.150 ohm) also cuts the series drop feeding the
LEDs, improving finding F1's own worst case from 8.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
Parts:
- added D44: SS14, Diode_SMD:D_SMA_Handsoldering, symbol Diode:SS14
- F4: value 1206L050/15YR -> 1206L110-C
Connections:
- net +12V: no longer F1.1
- net FAN_12V: now also D44.1 (K); no longer F1.2
- net P12_RAW: now also F1.1
- new net FAN_12V_RAW: D44.2 (A), F1.2
