File: hardware/breakout/sheets/analog-frontend.kicad_sch (KiCad schematic)
At the start: 128 parts, among them J19 ACCES I/O USB-AO16-8A mating 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, J20 Photodiode 1 (passive, coax, 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, J21 Photodiode 2 (passive, coax, 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, J22 Microphone (battery-powered, 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, J23 Ambient light sensor (battery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, J24 Accelerometer motion energy (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, J25 Joystick X (battery-powered, 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, J26 Joystick Y (battery-powered, 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, J27 Misc analog input 1 (panel BN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, J28 Misc analog input 1 (panel BN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, J29 Misc analog input 2 (panel BN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, J30 Misc analog input 2 (panel BN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, J31 Misc analog input 3 (panel BN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, J32 Misc analog input 3 (panel BN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, U16 INA105KU, U17 INA105KU, U18 INA105KU, U19 INA105KU, U20 INA105KU, U21 INA105KU, U22 OPA2197IDR, U23 OPA4197IDR, U24 INA105KU, U25 INA105KU, U26 INA105KU, U27 INA105KU, U28 INA105KU, U29 INA105KU, U30 INA105KU

Commit message: fix(hw): symmetric /1//2 divider on MISC1-3's shield leg
The MISC1-3 divider attenuated only the signal leg into INA105 "+",
leaving the shield leg (into "-") undivided. /1 mode cancelled the
shield disturbance correctly, but /2 mode output Vsig/2 - Vshield/2:
half the shield disturbance leaked through uncancelled, since a
difference amplifier only rejects common mode when both legs see the
same gain.

Mirrors the divider onto the shield leg (new _atten_leg() helper, same
matched 10.0k 0.1% resistors, same 3-pin jumper topology) so /2 mode
now divides both legs equally and Vshield cancels in both jumper
positions. Keeps the original before-the-amplifier placement and CMR
reasoning -- the "-" leg's own swing only shrinks relative to the
already-reviewed design, never grows.

The existing checker verified topology per leg but never compared the
two legs' own attenuation, approving the asymmetry vacuously. Adds
check_misc_leg_symmetry() (leg-fed-by-own-divider-common, matched
resistor values, genuine per-leg jumper topology) with two negative
controls, and fixes two of its own sibling checks whose assumptions
the new shield-leg structure broke (_check_bnc_shell_bonds' J-ref
count, _check_no_direct_agnd_reference's expected reference net) plus
one latent self-test ambiguity the new resistor exposed.

ERC: 0 errors, 31 warnings, byte-identical violation set to 4ecae2f.
All 5 project checkers (analog-frontend, power, taskpc-digital,
pi-interface, mule) pass with self-tests firing.

Co-Authored-By: Claude Opus 5 (1M context) <noreply@anthropic.com>
Parts:
- removed J29: Misc analog input 2 (panel BNC, /1//2 selectable), Connector_Coaxial:BNC_PanelMountable_Vertical, symbol Connector:Conn_Coaxial
- removed J30: Misc analog input 2 (panel BNC, /1//2 selectable)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, Connector_PinHeader_2.54mm:PinHeader_1x03_P2.54mm_Vertical, symbol Connector_Generic:Conn_01x03
- removed J31: Misc analog input 3 (panel BNC, /1//2 selectable), Connector_Coaxial:BNC_PanelMountable_Vertical, symbol Connector:Conn_Coaxial
- added J29: Misc analog input 1 (panel BNC, /1//2 selectable)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, Connector_PinHeader_2.54mm:PinHeader_1x03_P2.54mm_Vertical, symbol Connector_Generic:Conn_01x03
- added J30: Misc analog input 2 (panel BNC, /1//2 selectable), Connector_Coaxial:BNC_PanelMountable_Vertical, symbol Connector:Conn_Coaxial
- added J31: Misc analog input 2 (panel BNC, /1//2 selectable)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, Connector_PinHeader_2.54mm:PinHeader_1x03_P2.54mm_Vertical, symbol Connector_Generic:Conn_01x03
- added J33: Misc analog input 3 (panel BNC, /1//2 selectable), Connector_Coaxial:BNC_PanelMountable_Vertical, symbol Connector:Conn_Coaxial
- added J34, J35: Misc analog input 3 (panel BNC, /1//2 selectable)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, Connector_PinHeader_2.54mm:PinHeader_1x03_P2.54mm_Vertical, symbol Connector_Generic:Conn_01x03
- added R72: 1k, Resistor_SMD:R_0603_1608Metric, symbol Device:R
- added R73: 10, Resistor_SMD:R_0603_1608Metric, symbol Device:R
- added R74, R75, R76, R77: 10.0k 0.1%, Resistor_SMD:R_0603_1608Metric, symbol Device:R
- J28: value Misc analog input 1 (panel BNC, /1//2 selectable) -- shunt jumper: bridge 1-2 for x1 (clamp node direct), 2-3 for x2 (d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 -> Misc analog input 1 (panel BNC, /1//2 selectable) -- SIGNAL leg shunt jumper: bridge 1-2 for x1 (direct), 2-3 for x2 (d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
- J32: value Misc analog input 3 (panel BNC, /1//2 selectable) -- shunt jumper: bridge 1-2 for x1 (clamp node direct), 2-3 for x2 (d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 -> Misc analog input 2 (panel BNC, /1//2 selectable) -- SHIELD leg shunt jumper: bridge 1-2 for x1 (direct), 2-3 for x2 (d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
- R62, R63, R70, R71: value 10.0k -> 10.0k 0.1%
- R64, R68: value 1k -> 10.0k 0.1%
- R65, R69: value 10 -> 10.0k 0.1%
- R66: value 10.0k -> 1k
- R67: value 10.0k -> 10
Connections:
- net AGND: now also R73.2, R75.2, R77.2
- net A_MISC1_SHLD: now also R64.1, J29.1 (Pin_1); no longer U28.2 (-)
- net A_MISC2_CLAMP: now also R66.2, R68.1, J31.1 (Pin_1); no longer R64.2, R66.1
- net A_MISC2_DIV: now also J31.2 (Pin_2)
- net A_MISC2_MID: now also R68.2, R69.1, J31.3 (Pin_3); no longer R66.2, R67.1
- net A_MISC2_RAW: now also R66.1, J30.1 (In); no longer R64.1
- net A_MISC2_SHLD: now also J32.1 (Pin_1), R67.1, R70.1, J30.2 (Ext); no longer R65.1, U29.2 (-)
- net A_MISC3_CLAMP: now also J34.1 (Pin_1), R72.2, R74.1; no longer J32.1 (Pin_1), R68.2, R70.1
- net A_MISC3_DIV: now also J34.2 (Pin_2); no longer J32.2 (Pin_2)
- net A_MISC3_MID: now also J34.3 (Pin_3), R74.2, R75.1; no longer J32.3 (Pin_3), R70.2, R71.1
- net A_MISC3_RAW: now also J33.1 (In), R72.1; no longer R68.1
- net A_MISC3_SHLD: now also J33.2 (Ext), J35.1 (Pin_1), R73.1, R76.1; no longer R69.1, U30.2 (-)
- new net A_MISC1_SHLD_DIV: J29.2 (Pin_2), U28.2 (-)
- new net A_MISC1_SHLD_MID: J29.3 (Pin_3), R64.2, R65.1
- new net A_MISC2_SHLD_DIV: J32.2 (Pin_2), U29.2 (-)
- new net A_MISC2_SHLD_MID: J32.3 (Pin_3), R70.2, R71.1
- new net A_MISC3_SHLD_DIV: J35.2 (Pin_2), U30.2 (-)
- new net A_MISC3_SHLD_MID: J35.3 (Pin_3), R76.2, R77.1
Other:
- note added: "(fix round 1 -- task-10a-report.md: dividing the signal leg alone left half the"
- note added: "Both dividers sit BEFORE the amplifier: INA105's own linear common-mode range"
- note added: "THE TWO JUMPERS (signal leg, shield leg) MUST BE SET TO THE SAME POSITION -- a"
- note added: "does not want a raw +-10V swing directly."
- note added: "here and the bridge is left to the physical shunt (silkscreen/assembly note)."
- note added: "inputs additionally accept +-10V via switchable /1//2 attenuation, on BOTH legs"
- note added: "level electrical fact, so all header pins are wired to their own distinct nets"
- note added: "physical/assembly discipline, like the jumper position itself, not something"
- note added: "pin (2, wired to the amplifier) is bridged by a physical shunt jumper to EITHER"
- note added: "pin 1 (direct = /1) OR pin 3 (the /2 tap) at assembly time -- not a schematic-"
- note added: "resistors forming a fixed /2 tap to AGND, and its OWN 3-pin header whose common"
- note added: "shield = shield node) gets its OWN matched pair of ALWAYS-PRESENT 10.0k 0.1%"
- note added: "shield disturbance uncancelled in /2 mode). Each leg (signal = clamp node,"
- note added: "this schematic enforces; both headers' own description text repeats this."
- note removed: "/2 tap) at assembly time -- not a schematic-level electrical fact, so all three"
- note removed: "3-pin header's own common pin (2, the one wired to the amplifier) is bridged by"
- note removed: "PRESENT 10.0k resistors form a fixed /2 tap between the clamp node and AGND; a"
- note removed: "a physical shunt jumper to EITHER pin 1 (clamp node direct = /1) OR pin 3 (the"
- note removed: "header pins are wired to their own distinct nets here and the bridge is left to"
- note removed: "inputs additionally accept +-10V via switchable /1//2 attenuation. Two ALWAYS-"
- note removed: "places). Divider sits BEFORE the amplifier: INA105's own linear common-mode"
- note removed: "range does not want a raw +-10V swing directly."
- note removed: "the physical shunt (silkscreen/assembly note, not a component this generator"

Commit message: fix(hw): gang MISC1-3's /1//2 jumpers onto one physically-inseparable header
analog-frontend.kicad_sch (Task 10a fix round 1) gave each of MISC1-3's signal and shield
legs its own independent Conn_01x03 shunt header, both required to be set to the same
position but with nothing stopping them from disagreeing -- a field-reconfiguration risk
a reviewer flagged: years from now, someone changes a channel's range and forgets the
second jumper, silently re-creating the exact half-cancelled-shield-disturbance defect
fix round 1 closed out (the two-headers version left this as an explicitly-named residual
risk in its own docstring, judged at the time as "more component-library risk than this
fix warrants").

Replaces the two independent Conn_01x03 headers with one Conn_02x03_Top_Bottom header
(already in the Connector_Generic family this sheet already uses -- no new symbol or
footprint) carrying both legs: row 1 (pins 1-3) = signal, row 2 (pins 4-6) = shield.
Populated with a single 2-gang shorting block spanning both rows at the same column
position, both legs' jumper positions are now the same physical part -- disagreement is a
structural impossibility, not an assembly-discipline hope.

check_breakout_analog_frontend_netlist.py's _check_header_pin_roles() generalized to take
per-leg pin numbers (was hardcoded 1/2/3); _check_misc_leg_symmetry() now additionally
asserts both legs' own headers resolve to the SAME component reference, with a negative
control that relabels one leg's header pins onto a fake second ref and confirms the check
fires. All prior self-tests preserved unmodified in substance.

ERC: 0 errors, 22 warnings, unchanged from before this fix (no net contract changed, only
which physical part implements the jumper). check_breakout_power_netlist.py,
check_taskpc_digital_netlist.py, check_breakout_pi_interface_netlist.py, and
check_mule_netlist.py all re-run end to end and pass unaffected.

Co-Authored-By: Claude Opus 5 (1M context) <noreply@anthropic.com>
Parts:
- removed J28, J29: Misc analog input 1 (panel BNC, /1//2 selectable)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, Connector_PinHeader_2.54mm:PinHeader_1x03_P2.54mm_Vertical, symbol Connector_Generic:Conn_01x03
- removed J30: Misc analog input 2 (panel BNC, /1//2 selectable), Connector_Coaxial:BNC_PanelMountable_Vertical, symbol Connector:Conn_Coaxial
- removed J31, J32: Misc analog input 2 (panel BNC, /1//2 selectable)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, Connector_PinHeader_2.54mm:PinHeader_1x03_P2.54mm_Vertical, symbol Connector_Generic:Conn_01x03
- removed J33: Misc analog input 3 (panel BNC, /1//2 selectable), Connector_Coaxial:BNC_PanelMountable_Vertical, symbol Connector:Conn_Coaxial
- removed J34, J35: Misc analog input 3 (panel BNC, /1//2 selectable)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, Connector_PinHeader_2.54mm:PinHeader_1x03_P2.54mm_Vertical, symbol Connector_Generic:Conn_01x03
- added J28: Misc analog input 1 (panel BNC, /1//2 selectable)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, Connector_PinHeader_2.54mm:PinHeader_2x03_P2.54mm_Vertical, symbol Connector_Generic:Conn_02x03_Top_Bottom
- added J29: Misc analog input 2 (panel BNC, /1//2 selectable), Connector_Coaxial:BNC_PanelMountable_Vertical, symbol Connector:Conn_Coaxial
- added J30: Misc analog input 2 (panel BNC, /1//2 selectable)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, Connector_PinHeader_2.54mm:PinHeader_2x03_P2.54mm_Vertical, symbol Connector_Generic:Conn_02x03_Top_Bottom
- added J31: Misc analog input 3 (panel BNC, /1//2 selectable), Connector_Coaxial:BNC_PanelMountable_Vertical, symbol Connector:Conn_Coaxial
- added J32: Misc analog input 3 (panel BNC, /1//2 selectable)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, Connector_PinHeader_2.54mm:PinHeader_2x03_P2.54mm_Vertical, symbol Connector_Generic:Conn_02x03_Top_Bottom
Connections:
- net A_MISC1_CLAMP: now also J28.1 (Pin_1)
- net A_MISC1_DIV: now also J28.2 (Pin_2)
- net A_MISC1_MID: now also J28.3 (Pin_3)
- net A_MISC1_SHLD: now also J28.4 (Pin_4)
- net A_MISC1_SHLD_DIV: now also J28.5 (Pin_5)
- net A_MISC1_SHLD_MID: now also J28.6 (Pin_6)
- net A_MISC2_CLAMP: now also J30.1 (Pin_1)
- net A_MISC2_DIV: now also J30.2 (Pin_2)
- net A_MISC2_MID: now also J30.3 (Pin_3)
- net A_MISC2_RAW: now also J29.1 (In)
- net A_MISC2_SHLD: now also J29.2 (Ext), J30.4 (Pin_4)
- net A_MISC2_SHLD_DIV: now also J30.5 (Pin_5)
- net A_MISC2_SHLD_MID: now also J30.6 (Pin_6)
- net A_MISC3_CLAMP: now also J32.1 (Pin_1)
- net A_MISC3_DIV: now also J32.2 (Pin_2)
- net A_MISC3_MID: now also J32.3 (Pin_3)
- net A_MISC3_RAW: now also J31.1 (In)
- net A_MISC3_SHLD: now also J31.2 (Ext), J32.4 (Pin_4)
- net A_MISC3_SHLD_DIV: now also J32.5 (Pin_5)
- net A_MISC3_SHLD_MID: now also J32.6 (Pin_6)
Other:
- note added: "Conn_02x03 HEADER, populated with a SINGLE 2-GANG SHORTING BLOCK spanning both"
- note added: "FIX ROUND 2 (task-10b-report.md): both legs' own COMMON node (wired to the"
- note added: "OR the /2 tap (/2) at assembly/field-reconfiguration time -- not a schematic-"
- note added: "amplifier) is bridged by a physical shunt to EITHER the raw node (direct = /1)"
- note added: "and the bridge is left to the physical shunt. BOTH LEGS NOW SHARE ONE PHYSICAL"
- note added: "just against instructions) for the two legs to disagree: a real risk years from"
- note added: "leg pins 4-6; bridge 1-2+4-5 for x1, 2-3+5-6 for x2) -- replacing fix round 1's"
- note added: "level electrical fact, so every header pin is wired to its own distinct net here"
- note added: "now when someone reconfigures a channel's range and forgets the second jumper,"
- note added: "own two INDEPENDENT Conn_01x03 headers, which left it physically possible (not"
- note added: "resistors forming a fixed /2 tap to AGND."
- note added: "round 1 closed out. NEVER populate this header with two independent 1-gang"
- note added: "rows at the same column position (row 1 = signal leg pins 1-3, row 2 = shield"
- note added: "shunts -- that reintroduces the identical defect on a 2-row footprint."
- note added: "silently re-creating the exact half-cancelled-shield-disturbance defect fix"
- note removed: "THE TWO JUMPERS (signal leg, shield leg) MUST BE SET TO THE SAME POSITION -- a"
- note removed: "here and the bridge is left to the physical shunt (silkscreen/assembly note)."
- note removed: "level electrical fact, so all header pins are wired to their own distinct nets"
- note removed: "physical/assembly discipline, like the jumper position itself, not something"
- note removed: "pin (2, wired to the amplifier) is bridged by a physical shunt jumper to EITHER"
- note removed: "pin 1 (direct = /1) OR pin 3 (the /2 tap) at assembly time -- not a schematic-"
- note removed: "resistors forming a fixed /2 tap to AGND, and its OWN 3-pin header whose common"
- note removed: "this schematic enforces; both headers' own description text repeats this."

Commit message: fix(hw): correct MISC1-3 jumper pin map to match its real footprint geometry
665f211 ganged MISC1-3's /1//2 attenuator jumper onto one Conn_02x03_Top_Bottom header,
row 1 (pins 1-3) = signal leg, row 2 (pins 4-6) = shield leg, reasoning -- confirmed
"directly against the raw Connector_Generic library text" -- that pin N and pin N+3 share
a physical column. That confirmation checked the SCHEMATIC SYMBOL's own drawn geometry,
not the FOOTPRINT (PinHeader_2x03_P2.54mm_Vertical) actually assigned via footprint=, and
nothing in this toolchain cross-checks the two: kicad_sch.py's extract_symbol()/
unit_pins() reads only the .kicad_sym, never the .kicad_mod a symbol is paired with.

Rendered the real .kicad_mod (kicad-cli fp export svg) and read its pad coordinates
directly (both by hand and via hardware/gen/kicad_pcb.py's own footprint_pads(), already
built for the PCB-layout generator but never wired into any schematic-side check): the
real part is COLUMN-paired, not row-paired -- pads (1,2)/(3,4)/(5,6) sit 2.54mm apart (the
header's own minimum pitch), while (1,4)/(2,5)/(3,6), the pairing the shipped assignment
needed, sit 3.59mm apart on the diagonal. Under the shipped assignment, no shunt position
on the real part achieved "both legs at the same tap": pins 1-2 (genuinely adjacent) are
both RAW nodes, and pin 3 (signal DIV) sits nowhere near pin 4 (shield DIV) -- every
reachable position left one leg's own INA105 input floating, worse than the asymmetric-
divider defect this ganging change was made to prevent. Invisible to ERC and to every
netlist-topology checker in this project by construction: all of them reason about
electrical connectivity, and physical pad adjacency isn't a connectivity fact -- that is
the entire point of a jumper header.

Fixed by swapping the symbol, not the footprint: Conn_02x03_Odd_Even with pins assigned
INTERLEAVED (pin1=sig_raw, pin2=shld_raw, pin3=sig_div, pin4=shld_div, pin5=sig_mid,
pin6=shld_mid) instead of by row -- column A (pins 1,3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
Parts:
- removed J28: Misc analog input 1 (panel BNC, /1//2 selectable)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, Connector_PinHeader_2.54mm:PinHeader_2x03_P2.54mm_Vertical, symbol Connector_Generic:Conn_02x03_Top_Bottom
- removed J30: Misc analog input 2 (panel BNC, /1//2 selectable)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, Connector_PinHeader_2.54mm:PinHeader_2x03_P2.54mm_Vertical, symbol Connector_Generic:Conn_02x03_Top_Bottom
- removed J32: Misc analog input 3 (panel BNC, /1//2 selectable)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, Connector_PinHeader_2.54mm:PinHeader_2x03_P2.54mm_Vertical, symbol Connector_Generic:Conn_02x03_Top_Bottom
- added J28: Misc analog input 1 (panel BNC, /1//2 selectable)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, Connector_PinHeader_2.54mm:PinHeader_2x03_P2.54mm_Vertical, symbol Connector_Generic:Conn_02x03_Odd_Even
- added J30: Misc analog input 2 (panel BNC, /1//2 selectable)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, Connector_PinHeader_2.54mm:PinHeader_2x03_P2.54mm_Vertical, symbol Connector_Generic:Conn_02x03_Odd_Even
- added J32: Misc analog input 3 (panel BNC, /1//2 selectable)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, Connector_PinHeader_2.54mm:PinHeader_2x03_P2.54mm_Vertical, symbol Connector_Generic:Conn_02x03_Odd_Even
Connections:
- net A_MISC1_CLAMP: now also J28.1 (Pin_1)
- net A_MISC1_DIV: now also J28.3 (Pin_3)
- net A_MISC1_MID: now also J28.5 (Pin_5)
- net A_MISC1_SHLD: now also J28.2 (Pin_2)
- net A_MISC1_SHLD_DIV: now also J28.4 (Pin_4)
- net A_MISC1_SHLD_MID: now also J28.6 (Pin_6)
- net A_MISC2_CLAMP: now also J30.1 (Pin_1)
- net A_MISC2_DIV: now also J30.3 (Pin_3)
- net A_MISC2_MID: now also J30.5 (Pin_5)
- net A_MISC2_SHLD: now also J30.2 (Pin_2)
- net A_MISC2_SHLD_DIV: now also J30.4 (Pin_4)
- net A_MISC2_SHLD_MID: now also J30.6 (Pin_6)
- net A_MISC3_CLAMP: now also J32.1 (Pin_1)
- net A_MISC3_DIV: now also J32.3 (Pin_3)
- net A_MISC3_MID: now also J32.5 (Pin_5)
- net A_MISC3_SHLD: now also J32.2 (Pin_2)
- net A_MISC3_SHLD_DIV: now also J32.4 (Pin_4)
- net A_MISC3_SHLD_MID: now also J32.6 (Pin_6)
Other:
- note added: "'both legs at the same tap'. Symbol changed to Conn_02x03_Odd_Even, pins now"
- note added: "(divider tap) -- STILL NEVER two independent 1-gang shunts."
- note added: "1-gang shunts -- that reintroduces the identical defect on a 2-column footprint."
- note added: "Conn_02x03 HEADER, populated with a SINGLE 2-GANG SHORTING BLOCK -- replacing"
- note added: "FIX ROUND 3 (task-10b-report.md, this round): fix round 2's own PIN ASSIGNMENT"
- note added: "INTERLEAVED: column A (pins 1,3,5) = SIGNAL raw/div/mid, column B (pins 2,4,6) ="
- note added: "SHIELD raw/div/mid. Bridge pins 1-3 + 2-4 for x1 (direct), pins 3-5 + 4-6 for x2"
- note added: "assumed the wrong physical geometry for the real PinHeader_2x03_P2.54mm_Vertical"
- note added: "defect fix round 1 closed out. NEVER populate this header with two independent"
- note added: "fix round 1's own two INDEPENDENT Conn_01x03 headers, which left it physically"
- note added: "footprint (row-paired, pin N adjacent to pin N+3) -- the real part is COLUMN-"
- note added: "footprint_pads()), which left NO shunt position on the real part achieving"
- note added: "paired instead (confirmed via kicad-cli fp export svg + kicad_pcb.py's own"
- note added: "possible (not just against instructions) for the two legs to disagree: a real"
- note added: "risk years from now when someone reconfigures a channel's range and forgets the"
- note added: "second jumper, silently re-creating the exact half-cancelled-shield-disturbance"
- note removed: "Conn_02x03 HEADER, populated with a SINGLE 2-GANG SHORTING BLOCK spanning both"
- note removed: "just against instructions) for the two legs to disagree: a real risk years from"
- note removed: "leg pins 4-6; bridge 1-2+4-5 for x1, 2-3+5-6 for x2) -- replacing fix round 1's"
- note removed: "now when someone reconfigures a channel's range and forgets the second jumper,"
- note removed: "own two INDEPENDENT Conn_01x03 headers, which left it physically possible (not"
- note removed: "round 1 closed out. NEVER populate this header with two independent 1-gang"
- note removed: "rows at the same column position (row 1 = signal leg pins 1-3, row 2 = shield"
- note removed: "shunts -- that reintroduces the identical defect on a 2-row footprint."
- note removed: "silently re-creating the exact half-cancelled-shield-disturbance defect fix"
