File: hardware/breakout/sheets/opto-ni.kicad_sch (KiCad schematic)
At the start: 74 parts, among them J45 Connector 1 (digital, recordi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, U56 ACSL-6400-00TE, U57 ACSL-6400-00TE, U58 ACSL-6400-00TE, U59 ACSL-6400-00TE, U60 ACSL-6400-00TE, U61 ACSL-6400-00TE, U62 TMA-0505S

Commit message: fix(hw): drop opto-ni's NI-side pull-ups to 3.9k, within ACSL-6400's own RL-max
The original 10k pull-up (Task 11) was derived only by comparing against the
mule board's 1k -- it never checked ACSL-6400's own datasheet pull-up maximum
(RL-max = 4k, "Recommended Operating Conditions"), which it exceeded. 3.9k
(E24) is the largest standard value at or under that limit: still comfortably
inside NI's 250mA/connector budget (domain total 151-199mA, 51-99mA headroom,
vs 10k's 132-180mA bought only by violating the part's own spec), and the
edge-rate cost either way (tau ~0.2us at 3.9k vs ~0.5us at 10k, into ~50pF)
was never close enough to the 500us strobe period to be the deciding factor.
HIGH-level noise margin actually improves (worst-case VOH >= NI_5V-0.39V,
versus 10k's own -1.0V figure).

gen_breakout_opto_ni.py and check_breakout_opto_ni_netlist.py both move to
3.9k; opto-ni.kicad_sch regenerated (all 24 pull-ups). hardware/README.md
updated to match. The checker's own drift-to-1k negative control still fires
(relabeled to the new correct value, not weakened).

Also adds a general structural guard to check_breakout_opto_ni_netlist.py's
existing coordinate-collision scan: every same-column pair of real, placed
2-pin parts (vertical ones -- a part whose own two pins land on different X
columns, e.g. a coax jack's center/shield, is a different geometry and is
excluded rather than force-fit) must have disjoint pin-to-pin reach
intervals, derived from each part's own real library pin geometry rather
than only catching an actual duplicate label coordinate after the fact. This
is the third distinct instance of that defect class on this project
(analog-frontend's decoupling-cap short, task-10a-report.md; this sheet's own
NI_5V/channel-data-net short, CH_ROW_DY's own account in
gen_breakout_opto_ni.py) -- generalizes CH_ROW_DY's own "> Device:R's own
7.62mm span" comment into an executable, self-testing check instead of a
comment other generators have to remember to imitate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
Parts:
- R123, R125, R127, R129, R131, R133, R135, R137, R139, R141, R143, R145, R147, R149, R151, R153, R155, R157, R159, R161, R163, R165, R167, R169: value 10k -> 3.9k
Other:
- note added: "250mA budget; 3.9k pull-ups add ~31mA (domain total 151-199mA, 51-99mA"
- note added: "Logic-level integrity holds (worst-case VOH >= NI_5V-0.39V at the datasheet's"
- note added: "NI-SIDE PULL-UP: 3.9k -- fix round 1, corrected from this task's original 10k,"
- note added: "at or under that limit. 24 stages at ~5-7mA (IDDL) draw 120-168mA against NI's"
- note added: "decide this either way -- see the module docstring for the full derivation."
- note added: "headroom) -- 10k added only ~12mA, but only by violating the part's own spec."
- note added: "own datasheet RL-max (4k); 10k exceeded it. 3.9k (E24) is the largest E24 value"
- note added: "own worst-case leakage; VOL only improves at the lighter sink current); edge"
- note added: "rate (tau~0.2us into ~50pF) was never close enough to the 500us strobe to"
- note added: "which compared only against the mule's own 1k and never checked ACSL-6400's"
- note removed: "100uA leakage; VOL improves, not worsens, at 10k's lighter sink current) -- see"
- note removed: "15 MBd/5-TTL-load speed spec this sheet's real load -- a single high-Z NI DAQ"
- note removed: "1k. 24 output stages at ~5-7mA (ACSL-6400's own IDDL) is already 120-170mA"
- note removed: "NI-SIDE PULL-UP: 10k, per this task's own explicit instruction -- NOT the mule's"
- note removed: "against NI's 250mA/connector budget; 1k pull-ups add ~120mA more (near the"
- note removed: "input, hundreds-of-microseconds timing -- does not need); logic-level integrity"
- note removed: "is unaffected (worst-case VOH >= NI_5V-1.0V at the datasheet's own worst-case"
- note removed: "limit), 10k adds ~12mA. This EXCEEDS ACSL-6400's own datasheet RL-max (4k, a"
- note removed: "this generator's own module docstring for the full numeric derivation."

Commit message: fix(hw): one optocoupler LED per driver pin
The _BUF bank names 19 signals for what is really a 30-LED board. The 11
unnamed LEDs got doubled onto pins that already had one, and put +5V on
two sync-module GPIOs.

(a) Doubled loads. Each ACSL-6400/6420 LED draws ~7.33mA from +5V through
430R -- a value pinned between the part's 7-15mA recommended band and its
7.0mA worst-case switching threshold, so it cannot be lowered to suit a
driver. EVT_STROBE_BUF, RWD_CMD_BUF and STIM_TRIG_BUF each fed an NI LED
and an Intan LED from one HCT541 output (14.7mA vs 6mA IOL); BARCODE_PI
did the same off the pi-interface trigger buffer; and bare RWD_DLVR fed
both of its optocouplers straight off the 74HCT32 reward-OR gate, 14.7mA
against 4mA. That last one is the one with a failure mode rather than a
margin: RWD_DLVR's LOW is read by U14 (SN74LVC541APW, V_IL,max 0.8V), and
an HCT gate's VOL at 3.7x its rated sink plausibly exceeds it -- leaving
RWD_DLVR_PI stuck HIGH, the sync module recording reward-delivered
continuously. Same failure signature as the reward-OR polarity defect
caught on this board at task 8 fix round 1.

U10's 5 spare channels now carry EVT_STROBE_INTAN_BUF, RWD_CMD_INTAN_BUF,
STIM_TRIG_INTAN_BUF, RWD_DLVR_BUF and RWD_DLVR_INTAN_BUF (8 of 8 used);
U15's carry BARCODE_BUF and BARCODE_INTAN_BUF. The *_INTAN_BUF legs tap
the same *_CLAMP node their NI twin taps -- the established fan-out
point, one protection network with N buffered copies. RWD_DLVR and
BARCODE_PI now drive only CMOS inputs and panel headers.

(b) +5V reaching GPIO20/21 through an optocoupler LED. R166/R168 (430R
from +5V) fed ACSL-6400 LEDs whose cathodes sat on PD1_COMP/PD2_COMP --
which wire DIRECTLY into the sync module's GPIO20/21. With the LED off
that node idles ~3.6-3.8V, above the 3.3V rail and held only by the
module's ESD clamp; with this board powered and the sync box off, ~7mA is
injected into an unpowered pad. These were the only 2 of 24 NI
optocoupler LEDs not driven from a buffered le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
Connections:
- net BARCODE_PI renamed BARCODE_BUF
- net PD1_COMP renamed PD1_COMP_BUF
- net PD2_COMP renamed PD2_COMP_BUF
- net RWD_DLVR renamed RWD_DLVR_BUF

Commit message: fix(hardware): drive the optocoupler LEDs (F1, both halves)
430R never switched these LEDs. The original sizing solved
(5.0 - V_OL - V_F)/I correctly but against the rail's NOMINAL 5.00V and
V_F TYP; +5V reaches the anodes through F4 and D3 (0.42-0.49V of drop)
and V_F's worst case is 1.80V, so the real worst-case current was ~5mA
against the ACSL-6xx0's 7.0mA I_FH minimum. 30 channels were not
guaranteed to switch for seventy-three commits.

Both halves land together because neither is shippable alone -- 430R
starves the LED, and 249R (~12.7mA) overloads a single 7.5mA output.

Resistors, rail-aware: 430R -> 249R on the 30 LEDs fed from +5V, ->
301R on the 2 fed from ISO_5V. ISO_5V is regulated locally with nothing
in series, so 249R there would give 15.1mA -- past the 15mA ABSOLUTE
maximum. One value is wrong on one rail or the other.

Paralleling: every buffer-driven LED now has two SN74AHCT541 outputs
from tied inputs. Four new packages (U70-U73) plus C151-C154, 5 buffer
packages to 9, 6 spare channels. Channel maps are mirrored from the
tables that built the first leg rather than re-listed, so the legs
cannot drift apart. Refdes minted out of band, above the board maximum:
8 refs added, 0 removed, 0 renumbered.

This also fixes a per-PACKAGE limit no per-pin check could see. The
AHCT541's GND absolute maximum is 75mA (SCLS269Q 4.1, not the 100mA
hardware/README.md claimed); U8/U9 drive eight LEDs each; the drive is
active-low and the event bus idles at 0x0000, so sixteen LEDs are lit
CONTINUOUSLY. At 249R unparalleled that is ~101mA through one ground
pin. Paralleled it is 55.6mA worst case.

RHS_STIM_OUT's LED moves to a new buffered leg (RHS_STIM_OUT_BUF, off
U11's last two spare channels). It was the one channel driven by an
ACSL-6420 output rather than a buffer -- a deliberate, checked exception
that was correct at 430R (8.61mA of a 13mA budget) and not correct at
249R (13.85mA with its pull-up). The exception did not change; the
number it had been checked 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
Parts:
- R122, R124, R126, R128, R130, R132, R134, R136, R138, R140, R142, R144, R146, R148, R150, R152, R154, R156, R158, R160, R162, R164, R166, R168: value 430 -> 249
Connections:
- net RHS_STIM_OUT renamed RHS_STIM_OUT_BUF
Other:
- note added: "(AV02-0235EN footnote b) and of the 15mA ABSOLUTE maximum. 240R was rejected at"
- note added: "1.80V. 249R gives 8.6mA worst / 13.7mA best: clear of the 8mA guardbanded floor"
- note added: "1.95:1 against a 2.14:1 window, which fits with nothing to spare. That"
- note added: "7.0mA I_FH minimum, i.e. not guaranteed to switch at all. The original sizing"
- note added: "99% of that maximum; 270R misses the 8mA floor."
- note added: "LED DRIVE: 249R (E96, 1%) -- FINDING F1, 2026-08-16. Was 430R, which"
- note added: "THIS VALUE IS ONLY SAFE PARALLELED: at 249R one LED draws ~12.7mA, over a"
- note added: "external +5V supply is specified at +-2% -- at +-5% the tolerance spread is"
- note added: "outputs from tied inputs (taskpc-digital's U70-U73). It also assumes the"
- note added: "single SN74AHCT541 output's 7.5mA budget, so every LED here is driven by TWO"
- note added: "through F4 and D3 (0.38-0.45V of drop, so 4.55-4.62V) and VF's worst case is"
- note added: "tolerance is a load-bearing specification now, not an assumption."
- note added: "under-drove all 24 of these LEDs: ~5mA worst case against the ACSL-6xx0's own"
- note added: "using the rail's NOMINAL 5.00V and VF TYP (1.52V), but +5V reaches these anodes"
- note added: "was arithmetically right and physically wrong -- it solved (5.0V - VOL - VF)/I"
- note removed: "(E24) -> 7.33mA actual. Both VOL/VF figures are the closest datasheet test"
- note removed: "LED DRIVE: 430R (E24), targeting ~7.33mA -- roughly half ACSL-6400's own"
- note removed: "SN74HCT541 @ IOL=6mA) - VF(LED, 1.52V typ @ IF=10mA)) / 7.5mA = 420R -> 430R"
- note removed: "The timing budget is hundreds of microseconds, so the speed cost of a"
- note removed: "conservative drive is irrelevant; the CTR-degradation margin over a decade of"
- note removed: "datasheet-recommended top-of-range forward current (15mA/2=7.5mA), landing"
- note removed: "inside (not below) the recommended 7-15mA band. R = (5.0V - VOL(driver, 0.33V,"
- note removed: "points, used as approximations (flagged, not measured at this exact current)."
- note removed: "service is large."
