File: hardware/breakout/sheets/mux-intan.kicad_sch (KiCad schematic)
At the start: 64 parts, among them J37 Intan analog output 1 (BNC), J38 Intan analog output 2 (BNC), J39 Intan analog output 3 (BNC), J40 Intan analog output 4 (BNC), J41 Intan analog output 5 (BNC), J42 Intan analog output 6 (BNC), J43 Intan analog output 7 (BNC), J44 Intan analog output 8 (BNC), U38 ADG1206YRUZ, U39 INA105KU, U40 ADG1206YRUZ, U41 INA105KU, U42 ADG1206YRUZ, U43 INA105KU, U44 ADG1206YRUZ, U45 INA105KU, U46 ADG1206YRUZ, U47 INA105KU, U48 ADG1206YRUZ, U49 INA105KU, U50 ADG1206YRUZ, U51 INA105KU, U52 ADG1206YRUZ, U53 INA105KU

Commit message: fix(hw): replace ADG1206 A3 two-pin hedge with the real datasheet table
8fcba63 could not independently confirm the ADG1206YRUZ's physical pin for A3 on
the real 28-lead TSSOP (pin 13 vs. 14, 12+ fetch attempts, mostly blocked/timed
out) and, rather than guess silently, wired BOTH candidate pins to the same
MUX{n}_A3 net as a hedge. That was not a safe hedge: two different physical pins
tied to one net is a short between whatever those pins actually are, and would
have been a real fault, not a redundancy, had pin 13 turned out to be a supply or
a source pin instead of NC.

Replaced gen_wl_sync_lib.py's ADG1206_PINS with Table 4 of Analog Devices' own
ADG1206/ADG1207 Rev.0 datasheet, transcribed verbatim. This surfaced two more
errors the same hedge-era reconstruction carried: (1) it modelled TWO drain pins
(D1=28, D2=2, "tied together for 16:1 single-ended operation"), reasoning by
analogy from ADG1207's separate DA/DB pins on the shared silicon -- the real
ADG1206 brings out only ONE drain pin (D, pin 28); pin 2 is NC, not a second
output. (2) S9-S16's physical pin assignment was reversed (pin4->S9...pin11->S16
ascending, instead of Table 4's pin4->S16...pin11->S9 descending) -- would have
permuted 8 of the 16 A_* sources onto the wrong physical S-input on every one of
the 8 muxes had it shipped. gen_breakout_mux_intan.py updated to match: S9-S16
pin order corrected, MUX_PIN_D1/D2/A3_ALT collapsed to one MUX_PIN_D, the hedge
label removed, pins 2/3/13 left genuinely unconnected. Confirmed EN active-high
against the same table -- matches the existing design, no change needed there.
Recorded the full pin table, EN polarity, and address truth table (A3A2A1A0 =
0000 selects S1 ... 1111 selects S16, EN high throughout) in hardware/README.md
for Task 12.

Added two assertions to check_breakout_mux_intan_netlist.py, independent of the
generator's own choices, so a hedge of this kind cannot pass silently again:
_check_no_signal_pin_collisions() (no two of a mux's own 21 si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
Connections:
- net A_ACC: now also U38.10 (S10), U40.10 (S10), U42.10 (S10), U44.10 (S10), U46.10 (S10), U48.10 (S10), U50.10 (S10), U52.10 (S10); no longer U38.5 (S10), U40.5 (S10), U42.5 (S10), U44.5 (S10), U46.5 (S10), U48.5 (S10), U50.5 (S10), U52.5 (S10)
- net A_AMB: now also U38.11 (S9), U40.11 (S9), U42.11 (S9), U44.11 (S9), U46.11 (S9), U48.11 (S9), U50.11 (S9), U52.11 (S9); no longer U38.4 (S9), U40.4 (S9), U42.4 (S9), U44.4 (S9), U46.4 (S9), U48.4 (S9), U50.4 (S9), U52.4 (S9)
- net A_JOY_X: now also U38.9 (S11), U40.9 (S11), U42.9 (S11), U44.9 (S11), U46.9 (S11), U48.9 (S11), U50.9 (S11), U52.9 (S11); no longer U38.6 (S11), U40.6 (S11), U42.6 (S11), U44.6 (S11), U46.6 (S11), U48.6 (S11), U50.6 (S11), U52.6 (S11)
- net A_JOY_Y: now also U38.8 (S12), U40.8 (S12), U42.8 (S12), U44.8 (S12), U46.8 (S12), U48.8 (S12), U50.8 (S12), U52.8 (S12); no longer U38.7 (S12), U40.7 (S12), U42.7 (S12), U44.7 (S12), U46.7 (S12), U48.7 (S12), U50.7 (S12), U52.7 (S12)
- net A_MIC: now also U38.7 (S13), U40.7 (S13), U42.7 (S13), U44.7 (S13), U46.7 (S13), U48.7 (S13), U50.7 (S13), U52.7 (S13); no longer U38.8 (S13), U40.8 (S13), U42.8 (S13), U44.8 (S13), U46.8 (S13), U48.8 (S13), U50.8 (S13), U52.8 (S13)
- net A_MISC1: now also U38.6 (S14), U40.6 (S14), U42.6 (S14), U44.6 (S14), U46.6 (S14), U48.6 (S14), U50.6 (S14), U52.6 (S14); no longer U38.9 (S14), U40.9 (S14), U42.9 (S14), U44.9 (S14), U46.9 (S14), U48.9 (S14), U50.9 (S14), U52.9 (S14)
- net A_MISC2: now also U38.5 (S15), U40.5 (S15), U42.5 (S15), U44.5 (S15), U46.5 (S15), U48.5 (S15), U50.5 (S15), U52.5 (S15); no longer U38.10 (S15), U40.10 (S15), U42.10 (S15), U44.10 (S15), U46.10 (S15), U48.10 (S15), U50.10 (S15), U52.10 (S15)
- net A_MISC3: now also U38.4 (S16), U40.4 (S16), U42.4 (S16), U44.4 (S16), U46.4 (S16), U48.4 (S16), U50.4 (S16), U52.4 (S16); no longer U38.11 (S16), U40.11 (S16), U42.11 (S16), U44.11 (S16), U46.11 (S16), U48.11 (S16), U50.11 (S16), U52.11 (S16)
- net MUX1_A3: no longer U38.13 (A3_ALT_NC)
- net MUX2_A3: no longer U40.13 (A3_ALT_NC)
- net MUX3_A3: no longer U42.13 (A3_ALT_NC)
- net MUX4_A3: no longer U44.13 (A3_ALT_NC)
- net MUX5_A3: no longer U46.13 (A3_ALT_NC)
- net MUX6_A3: no longer U48.13 (A3_ALT_NC)
- net MUX7_A3: no longer U50.13 (A3_ALT_NC)
- net MUX8_A3: no longer U52.13 (A3_ALT_NC)
- net MUX_OUT1: no longer U38.2 (D2)
- net MUX_OUT2: no longer U40.2 (D2)
- net MUX_OUT3: no longer U42.2 (D2)
- net MUX_OUT4: no longer U44.2 (D2)
- net MUX_OUT5: no longer U46.2 (D2)
- net MUX_OUT6: no longer U48.2 (D2)
- net MUX_OUT7: no longer U50.2 (D2)
- net MUX_OUT8: no longer U52.2 (D2)
Other:
- note added: "(ALL_16_NETS/S_PIN_NUMBERS list order) -- like gen_breakout_analog_ni.py's"
- note added: "(S1-S16, D, EN, VDD/VSS/GND) is one of the 16 A_* nets, MUX_OUT{n}, or"
- note added: "A3 net rather than guess silently. That was not a safe hedge -- two different"
- note added: "Devices' own ADG1206/ADG1207 Rev.0 datasheet, 28-Lead TSSOP column,"
- note added: "NO HEDGE: the originally committed version of this symbol could not"
- note added: "PIN MAP, DEFINITIVE (fix round 1, task-10c-report.md): Table 4 of Analog"
- note added: "S1-S16/A0-A3 pin NAMES are the datasheet's own (Table 4, fix round 1,"
- note added: "S9) is still this sheet's own declared, arbitrary-but-fixed choice"
- note added: "always enabled -- selection is by address only). Each mux's own single D"
- note added: "are, and would have been a fault, not a redundancy, had pin 13 turned out to"
- note added: "be a supply or source pin instead of NC. This fix round replaced the hedge"
- note added: "blocked/timed out rather than conflicting) and wired BOTH pins to the same"
- note added: "for the full 28-pin table. A3 is pin 14. Pins 2, 3, and 13 are this part's"
- note added: "independently confirm pin 13 vs. 14 for A3 (12+ fetch attempts, mostly"
- note added: "only NC pins and carry no net on this sheet."
- note added: "output (pin 28, this part's own one common drain) feeds MUX_OUT{n} into one"
- note added: "own AI-channel-number assignment, no datasheet fixes a board's own source-"
- note added: "physical pins tied to one net is a short between whatever those pins actually"
- note added: "reach any of Intan's 8 channels. EN tied to +12V (active-high per Table 4,"
- note added: "selects S1 ... 1111 selects S16, EN high) is in hardware/README.md."
- note added: "selects the same relative source everywhere. Address truth table (0000"
- note added: "sheet's own labels awaiting a later task (10a's *_TPC, 10b's *_BUF). Address"
- note added: "sourced fact, not a choice. WHICH A_* source rides which mux pin (S1 vs."
- note added: "task-10c-report.md) -- physical pin 19 IS S1, physical pin 14 IS A3, a"
- note added: "throughout) is in hardware/README.md for Task 12."
- note added: "to-channel assignment. Same order used on all 8 muxes, so one address value"
- note added: "transcribed verbatim -- see gen_wl_sync_lib.py's own ADG1206YRUZ block comment"
- note added: "truth table (A3 A2 A1 A0 = 0000 selects S1 ... 1111 selects S16, EN high"
- note added: "with the real datasheet table above."
- note removed: "(S1-S16, D1/D2, EN, VDD/VSS/GND) is one of the 16 A_* nets, MUX_OUT{n}, or"
- note removed: "ADG1206YRUZ block comment for the full account. VERIFY AGAINST THE REAL"
- note removed: "ADG1207BCPZ stock symbol (same manufacturer family, same NC-cluster-before-"
- note removed: "DATASHEET OR A PHYSICAL SAMPLE BEFORE FABRICATION, same disclosure discipline"
- note removed: "PIN MAP CONFIDENCE, stated explicitly per this task's own instruction: pin"
- note removed: "S-type/address-type at all. Same order used on all 8 muxes, so one address"
- note removed: "S1-S16/A0-A3 index assignment (which A_* source rides which mux pin; which"
- note removed: "TSSOP-28 (pin 13 vs. 14) could not be independently confirmed despite"
- note removed: "address-cluster structure). The EXACT physical pin NUMBER for A3 on the real"
- note removed: "against multiple independent sources AND this project's own locally-installed"
- note removed: "arbitrary-but-fixed choice (ALL_16_NETS/S_PIN_NUMBERS list order) -- like"
- note removed: "as hardware/README.md's own mini-XLR/M12 footprint confidence table."
- note removed: "conflicting) -- hedged by wiring BOTH pins 13 and 14 to this design's own A3"
- note removed: "extensive effort (12+ fetch attempts, mostly blocked/timed out rather than"
- note removed: "gen_breakout_analog_ni.py's own AI-channel-number assignment, no external"
- note removed: "input if the reconstruction has it backwards). See gen_wl_sync_lib.py's own"
- note removed: "is by address only). Each mux's own D1/D2 output (tied together, this part's"
- note removed: "net (harmless if one is truly NC; protects against a floating real address"
- note removed: "own datasheet way to get 16:1 single-ended operation) feeds MUX_OUT{n} into one"
- note removed: "physical address pin is software's A0 vs. A3) is this sheet's own declared,"
- note removed: "reach any of Intan's 8 channels. EN tied to +12V (always enabled -- selection"
- note removed: "roles (16 S-type, 2 D-type, 4 address, EN, VDD/VSS/GND) are well-corroborated"
- note removed: "sheet's own labels awaiting a later task (10a's *_TPC, 10b's *_BUF)."
- note removed: "source fixes this the way a real datasheet fixes WHICH PHYSICAL PINS are"
- note removed: "value selects the same relative source everywhere."

Commit message: fix(hardware): the analog front-end corrections (F3, M1, M2, M4; D1 recorded)
Five findings, both photodiode channels each.

F3 -- THE TRANSIMPEDANCE STAGE SATURATED. R38/R40 1M -> 180k. An FDS100 is
13 mm2 at 0.30 A/W, so a display flip patch at ~0.29 mW/cm2 delivers
~11.3 uA -- and 11.3 uA x 1M demands 11.3 V, twice this board's +-5 V analog
convention and past both NI's and Intan's input range. The stage clipped
long before full scale.

That matters more than a gain error sounds. The flat part is the BRIGHT
part, and the edge these channels exist to time is what survives, so the
defect would have looked like "it works" on a scope. 180k puts peak white
near 2.0 V, which also lands inside the DAC's own 0-2.048 V span after D1.

The DNP parallel trim positions the finding asks for are fitted (R196/R197,
unpopulated). A resistor pad rather than a jumper, deliberately: gain rests
on an estimate of display irradiance rather than a measurement, so bring-up
needs a way to move it, but a mechanical contact at a 180k summing junction
would be a leakage and noise liability.

M1 -- IT WAS ALSO UNDER-COMPENSATED. C48/C50 3.3pF -> 22pF. 3.3pF was
fitted for a 1M stage against an assumed 300-500 pF of input capacitance.
Thorlabs publish the FDS100's capacitance only at 20 V bias (24 pF); this
design is forced into ZERO bias by the no-power-in-the-booth constraint,
where it is at maximum and unpublished -- estimated 130-380 pF, and 440-900
pF with 3-5 m of coax.

22pF at 180k is deliberate over-compensation, not a fit: stable to 5.5 nF
of input capacitance (~50 m of coax) at -3 dB = 40 kHz, still four times
what these channels need. The stage stops depending on cable length and on
a diode capacitance nobody can look up. The BOM now calls for C0G/NP0 on
these two rather than X7R -- a compensation capacitor whose value moves
with bias or temperature is not doing this job.

M2 -- THE MUX TAPPED THE WRONG NODE. The eight muxes' S7/S8 inputs move
from A_PD1/A_PD2 to A_PD1_NI_BUF/A_PD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
Connections:
- net A_PD1 renamed A_PD1_NI_BUF
- net A_PD2 renamed A_PD2_NI_BUF
Changed lines of the file:
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@@
 		)
 	)
-	(global_label "A_PD1"
+	(global_label "A_PD1_NI_BUF"
 		(shape bidirectional)
 		(at 20.320000000000004 16.509999999999998 0)
@@
 		)
 	)
-	(global_label "A_PD2"
+	(global_label "A_PD2_NI_BUF"
 		(shape bidirectional)
 		(at 20.320000000000004 19.05 0)
@@
 		)
 	)
-	(global_label "A_PD1"
+	(global_label "A_PD1_NI_BUF"
 		(shape bidirectional)
 		(at 20.320000000000004 80.00999999999999 0)
@@
 		)
 	)
-	(global_label "A_PD2"
+	(global_label "A_PD2_NI_BUF"
 		(shape bidirectional)
 		(at 20.320000000000004 82.55 0)
@@
 		)
 	)
-	(global_label "A_PD1"
+	(global_label "A_PD1_NI_BUF"
 		(shape bidirectional)
 		(at 20.320000000000004 143.51 0)
@@
 		)
 	)
-	(global_label "A_PD2"
+	(global_label "A_PD2_NI_BUF"
 		(shape bidirectional)
 		(at 20.320000000000004 146.04999999999998 0)
@@
 		)
 	)
-	(global_label "A_PD1"
+	(global_label "A_PD1_NI_BUF"
 		(shape bidirectional)
 		(at 20.320000000000004 207.01 0)
@@
 		)
 	)
-	(global_label "A_PD2"
+	(global_label "A_PD2_NI_BUF"
 		(shape bidirectional)
 		(at 20.320000000000004 209.54999999999998 0)
@@
 		)
 	)
-	(global_label "A_PD1"
+	(global_label "A_PD1_NI_BUF"
 		(shape bidirectional)
 		(at 20.320000000000004 270.51 0)
@@
 		)
 	)
-	(global_label "A_PD2"
+	(global_label "A_PD2_NI_BUF"
 		(shape bidirectional)
 		(at 20.320000000000004 273.05 0)
@@
 		)
 	)
-	(global_label "A_PD1"
+	(global_label "A_PD1_NI_BUF"
 		(shape bidirectional)
 		(at 20.320000000000004 334.01 0)
@@
 		)
 	)
-	(global_label "A_PD2"
+	(global_label "A_PD2_NI_BUF"
 		(shape bidirectional)
 		(at 20.320000000000004 336.55 0)
@@
 		)
 	)
-	(global_label "A_PD1"
+	(global_label "A_PD1_NI_BUF"
 		(shape bidirectional)
 		(at 20.320000000000004 397.51 0)
@@
 		)
 	)
-	(global_label "A_PD2"
+	(global_label "A_PD2_NI_BUF"
 		(shape bidirectional)
 		(at 20.320000000000004 400.05 0)
@@
 		)
 	)
-	(global_label "A_PD1"
+	(global_label "A_PD1_NI_BUF"
 		(shape bidirectional)
 		(at 20.320000000000004 461.01 0)
@@
 		)
 	)
-	(global_label "A_PD2"
+	(global_label "A_PD2_NI_BUF"
 		(shape bidirectional)
 		(at 20.320000000000004 463.55 0)
