File: hardware/breakout/sheets/mux-intan.kicad_sch (KiCad schematic)
At the start: 64 parts, among them J37 Intan analog output 1 (BNC), J38 Intan analog output 2 (BNC), J39 Intan analog output 3 (BNC), J40 Intan analog output 4 (BNC), J41 Intan analog output 5 (BNC), J42 Intan analog output 6 (BNC), J43 Intan analog output 7 (BNC), J44 Intan analog output 8 (BNC), U38 ADG1206YRUZ, U39 INA105KU, U40 ADG1206YRUZ, U41 INA105KU, U42 ADG1206YRUZ, U43 INA105KU, U44 ADG1206YRUZ, U45 INA105KU, U46 ADG1206YRUZ, U47 INA105KU, U48 ADG1206YRUZ, U49 INA105KU, U50 ADG1206YRUZ, U51 INA105KU, U52 ADG1206YRUZ, U53 INA105KU

Commit message: fix(hardware): rebuild the connectors on their primary drawings (F6, R1, D3)
Audit step 5, the mechanical half. Three connectors changed, one of them a
fab-stopper, and none of it was visible to the netlist.

MDR68 (the fab-stopper). Rebuilt from MH drawing 3700-0121-01 rev 3.0. The
as-built footprint drilled contacts at 0.5 mm against a required 0.85 mm -- the
pins do not fit, so the board could not have been assembled -- and laid them out
as 2 rows at 2.84 mm where the drawing shows 4 staggered rows of 17 at 1.905 mm.
The 4-row stagger is what makes an 0.85 mm drill manufacturable at a 1.27 mm
mating pitch at all; the array now spans the drawing's own 41.91 mm exactly,
which is the arithmetic that confirms the reading. The claim made during the
audit that it had "no mounting holes at all" was wrong: it had two, Ø2.79 on
57.9 mm centres against the drawing's Ø2.77 on 57.93.

M12 (ruling R1). M12A_5_Panel is deleted, symbol and footprint and generator
function alike. Its contact geometry was sourced well -- IEC 61076-2-101
A-coding, cross-checked three ways -- and it made no difference, because the part
the design procures (Phoenix 1551833) terminates in AWG 22-20 wire and mounts
through the panel. It has no PCB tails, so no board-mount footprint of any
dimensions could have been right, and as built every cable insertion and every
3-4 N.m tightening loaded PCB pads directly. J1 is now a stock 5-way header where
those flying leads land; the connector stays in the order BOM as chassis
furniture.

BNC (F6). BNC_PanelMountable_Vertical puts the connector axis perpendicular to
the PCB -- a 9.65 mm barrel hole through the board -- so on a 430x240 mm board
lying flat in a 2U chassis all 31 barrels pointed at the lid rather than at the
panels. It also cost 5,654 mm2 of pad and 2,267 mm2 of removed copper on every
layer. Replaced by a right-angle dual jack built from Amphenol drawing 31-6575
rev A: 31 ports on 17 bodies, 3 spare ports, every shell still routed
individually.
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
Parts:
- removed J37: Intan analog output 1 (BNC), Connector_Coaxial:BNC_PanelMountable_Vertical, symbol Connector:Conn_Coaxial
- removed J38: Intan analog output 2 (BNC), Connector_Coaxial:BNC_PanelMountable_Vertical, symbol Connector:Conn_Coaxial
- removed J39: Intan analog output 3 (BNC), Connector_Coaxial:BNC_PanelMountable_Vertical, symbol Connector:Conn_Coaxial
- removed J40: Intan analog output 4 (BNC), Connector_Coaxial:BNC_PanelMountable_Vertical, symbol Connector:Conn_Coaxial
- removed J41: Intan analog output 5 (BNC), Connector_Coaxial:BNC_PanelMountable_Vertical, symbol Connector:Conn_Coaxial
- removed J42: Intan analog output 6 (BNC), Connector_Coaxial:BNC_PanelMountable_Vertical, symbol Connector:Conn_Coaxial
- removed J43: Intan analog output 7 (BNC), Connector_Coaxial:BNC_PanelMountable_Vertical, symbol Connector:Conn_Coaxial
- removed J44: Intan analog output 8 (BNC), Connector_Coaxial:BNC_PanelMountable_Vertical, symbol Connector:Conn_Coaxial
- added J37: Dual panel BNC: Intan analog output 1 (BNC) | Int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, wl-sync:BNC_Dual_RA_Isolated, symbol wl-sync:BNC_Dual_RA_Isolated
- added J39: Dual panel BNC: Intan analog output 3 (BNC) | Int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, wl-sync:BNC_Dual_RA_Isolated, symbol wl-sync:BNC_Dual_RA_Isolated
- added J41: Dual panel BNC: Intan analog output 5 (BNC) | Int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, wl-sync:BNC_Dual_RA_Isolated, symbol wl-sync:BNC_Dual_RA_Isolated
- added J43: Dual panel BNC: Intan analog output 7 (BNC) | Int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, wl-sync:BNC_Dual_RA_Isolated, symbol wl-sync:BNC_Dual_RA_Isolated
Connections:
- net INTAN_AO1: now also J37.1 (A_In)
- net INTAN_AO2: now also J37.3 (B_In)
- net INTAN_AO3: now also J39.1 (A_In)
- net INTAN_AO4: now also J39.3 (B_In)
- net INTAN_AO5: now also J41.1 (A_In)
- net INTAN_AO6: now also J41.3 (B_In)
- net INTAN_AO7: now also J43.1 (A_In)
- net INTAN_AO8: now also J43.3 (B_In)
- net INTAN_GND: now also J37.2 (A_Ext), J37.4 (B_Ext), J39.2 (A_Ext), J39.4 (B_Ext), J41.2 (A_Ext), J41.4 (B_Ext), J43.2 (A_Ext), J43.4 (B_Ext)
Changed lines of the file:
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@@
 	)
 	(symbol
-		(lib_id "Connector:Conn_Coaxial")
+		(lib_id "wl-sync:BNC_Dual_RA_Isolated")
 		(at 175.26 20.32 0)
 		(unit 1)
@@
 			(effects (font (size 1.27 1.27)))
 		)
-		(property "Value" "Intan analog output 1 (BNC)"
+		(property "Value" "Dual panel BNC: Intan analog output 1 (BNC) | Intan analog output 2 (BNC)"
 			(at 177.292 22.86 0)
 			(effects (font (size 1.27 1.27)))
 		)
-		(property "Footprint" "Connector_Coaxial:BNC_PanelMountable_Vertical"
+		(property "Footprint" "wl-sync:BNC_Dual_RA_Isolated"
 			(at 175.26 20.32 0)
 			(effects (font (size 1.27 1.27)) (hide yes))
@@
 	)
 	(symbol
-		(lib_id "Connector:Conn_Coaxial")
+		(lib_id "wl-sync:BNC_Dual_RA_Isolated")
 		(at 175.26 83.82 0)
-		(unit 1)
+		(unit 2)
 		(exclude_from_sim no)
 		(in_bom yes)
 		(on_board yes)
 		(dnp no)
-		(property "Reference" "J38"
+		(property "Reference" "J37"
 			(at 177.292 83.82 0)
 			(effects (font (size 1.27 1.27)))
 		)
-		(property "Value" "Intan analog output 2 (BNC)"
+		(property "Value" "Dual panel BNC: Intan analog output 1 (BNC) | Intan analog output 2 (BNC)"
 			(at 177.292 86.36 0)
 			(effects (font (size 1.27 1.27)))
 		)
-		(property "Footprint" "Connector_Coaxial:BNC_PanelMountable_Vertical"
+		(property "Footprint" "wl-sync:BNC_Dual_RA_Isolated"
 			(at 175.26 83.82 0)
 			(effects (font (size 1.27 1.27)) (hide yes))
@@
 			(effects (font (size 1.27 1.27)) (hide yes))
 		)
-		(pin "1")
-		(pin "2")
+		(pin "3")
+		(pin "4")
 		(instances
 			(project "breakout"
 				(path "/d2c4d978-5db4-46d9-a1cd-a7af0aeb1700/9642e779-bb28-44cd-b82a-6706defd6bbc"
-					(reference "J38") (unit 1)
+					(reference "J37") (unit 2)
 				)
 			)
@@
 	)
 	(symbol
-		(lib_id "Connector:Conn_Coaxial")
+		(lib_id "wl-sync:BNC_Dual_RA_Isolated")
 		(at 175.26 147.32 0)
 		(unit 1)
@@
 			(effects (font (size 1.27 1.27)))
 		)
-		(property "Value" "Intan analog output 3 (BNC)"
+		(property "Value" "Dual panel BNC: Intan analog output 3 (BNC) | Intan analog output 4 (BNC)"
 			(at 177.292 149.85999999999999 0)
 			(effects (font (size 1.27 1.27)))
 		)
-		(property "Footprint" "Connector_Coaxial:BNC_PanelMountable_Vertical"
+		(property "Footprint" "wl-sync:BNC_Dual_RA_Isolated"
 			(at 175.26 147.32 0)
 			(effects (font (size 1.27 1.27)) (hide yes))
@@
 	)
 	(symbol
-		(lib_id "Connector:Conn_Coaxial")
+		(lib_id "wl-sync:BNC_Dual_RA_Isolated")
 		(at 175.26 210.82 0)
-		(unit 1)
+		(unit 2)
 		(exclude_from_sim no)
 		(in_bom yes)
 		(on_board yes)
 		(dnp no)
-		(property "Reference" "J40"
+		(property "Reference" "J39"
 			(at 177.292 210.82 0)
 			(effects (font (size 1.27 1.27)))
 		)
-		(property "Value" "Intan analog output 4 (BNC)"
+		(property "Value" "Dual panel BNC: Intan analog output 3 (BNC) | Intan analog output 4 (BNC)"
 			(at 177.292 213.35999999999999 0)
 			(effects (font (size 1.27 1.27)))
 		)
-		(property "Footprint" "Connector_Coaxial:BNC_PanelMountable_Vertical"
+		(property "Footprint" "wl-sync:BNC_Dual_RA_Isolated"
 			(at 175.26 210.82 0)
 			(effects (font (size 1.27 1.27)) (hide yes))
@@
 			(effects (font (size 1.27 1.27)) (hide yes))
 		)
-		(pin "1")
-		(pin "2")
+		(pin "3")
+		(pin "4")
 		(instances
 			(project "breakout"
 				(path "/d2c4d978-5db4-46d9-a1cd-a7af0aeb1700/9642e779-bb28-44cd-b82a-6706defd6bbc"
-					(reference "J40") (unit 1)
+					(reference "J39") (unit 2)
 				)
 			)
@@
 	)
 	(symbol
-		(lib_id "Connector:Conn_Coaxial")
+		(lib_id "wl-sync:BNC_Dual_RA_Isolated")
 		(at 175.26 274.32 0)
 		(unit 1)
@@
 			(effects (font (size 1.27 1.27)))
 		)
-		(property "Value" "Intan analog output 5 (BNC)"
+		(property "Value" "Dual panel BNC: Intan analog output 5 (BNC) | Intan analog output 6 (BNC)"
 			(at 177.292 276.86 0)
 			(effects (font (size 1.27 1.27)))
 		)
-		(property "Footprint" "Connector_Coaxial:BNC_PanelMountable_Vertical"
+		(property "Footprint" "wl-sync:BNC_Dual_RA_Isolated"
 			(at 175.26 274.32 0)
 			(effects (font (size 1.27 1.27)) (hide yes))
@@
 	)
 	(symbol
-		(lib_id "Connector:Conn_Coaxial")
+		(lib_id "wl-sync:BNC_Dual_RA_Isolated")
 		(at 175.26 337.82 0)
-		(unit 1)
+		(unit 2)
 		(exclude_from_sim no)
 		(in_bom yes)
 		(on_board yes)
 		(dnp no)
-		(property "Reference" "J42"
+		(property "Reference" "J41"
 			(at 177.292 337.82 0)
 			(effects (font (size 1.27 1.27)))
 		)
-		(property "Value" "Intan analog output 6 (BNC)"
+		(property "Value" "Dual panel BNC: Intan analog output 5 (BNC) | Intan analog output 6 (BNC)"
 			(at 177.292 340.36 0)
 			(effects (font (size 1.27 1.27)))
 		)
-		(property "Footprint" "Connector_Coaxial:BNC_PanelMountable_Vertical"
+		(property "Footprint" "wl-sync:BNC_Dual_RA_Isolated"
 			(at 175.26 337.82 0)
 			(effects (font (size 1.27 1.27)) (hide yes))
@@
 			(effects (font (size 1.27 1.27)) (hide yes))
 		)
-		(pin "1")
-		(pin "2")
+		(pin "3")
+		(pin "4")
 		(instances
 			(project "breakout"
 				(path "/d2c4d978-5db4-46d9-a1cd-a7af0aeb1700/9642e779-bb28-44cd-b82a-6706defd6bbc"
-					(reference "J42") (unit 1)
+					(reference "J41") (unit 2)
 				)
 			)
@@
 	)
 	(symbol
-		(lib_id "Connector:Conn_Coaxial")
+		(lib_id "wl-sync:BNC_Dual_RA_Isolated")
 		(at 175.26 401.32 0)
 		(unit 1)
@@
 			(effects (font (size 1.27 1.27)))
 		)
-		(property "Value" "Intan analog output 7 (BNC)"
+		(property "Value" "Dual panel BNC: Intan analog output 7 (BNC) | Intan analog output 8 (BNC)"
 			(at 177.292 403.86 0)
 			(effects (font (size 1.27 1.27)))
 		)
-		(property "Footprint" "Connector_Coaxial:BNC_PanelMountable_Vertical"
+		(property "Footprint" "wl-sync:BNC_Dual_RA_Isolated"
 			(at 175.26 401.32 0)
 			(effects (font (size 1.27 1.27)) (hide yes))
@@
 	)
 	(symbol
-		(lib_id "Connector:Conn_Coaxial")
+		(lib_id "wl-sync:BNC_Dual_RA_Isolated")
 		(at 175.26 464.82 0)
-		(unit 1)
+		(unit 2)
 		(exclude_from_sim no)
 		(in_bom yes)
 		(on_board yes)
 		(dnp no)
-		(property "Reference" "J44"
+		(property "Reference" "J43"
 			(at 177.292 464.82 0)
 			(effects (font (size 1.27 1.27)))
 		)
-		(property "Value" "Intan analog output 8 (BNC)"
+		(property "Value" "Dual panel BNC: Intan analog output 7 (BNC) | Intan analog output 8 (BNC)"
 			(at 177.292 467.36 0)
 			(effects (font (size 1.27 1.27)))
 		)
-		(property "Footprint" "Connector_Coaxial:BNC_PanelMountable_Vertical"
+		(property "Footprint" "wl-sync:BNC_Dual_RA_Isolated"
 			(at 175.26 464.82 0)
 			(effects (font (size 1.27 1.27)) (hide yes))
@@
 			(effects (font (size 1.27 1.27)) (hide yes))
 		)
-		(pin "1")
-		(pin "2")
+		(pin "3")
+		(pin "4")
 		(instances
 			(project "breakout"
 				(path "/d2c4d978-5db4-46d9-a1cd-a7af0aeb1700/9642e779-bb28-44cd-b82a-6706defd6bbc"
-					(reference "J44") (unit 1)
+					(reference "J43") (unit 2)
 				)
 			)
