File: hardware/breakout/sheets/comparators.kicad_sch (KiCad schematic)
At the start: 17 parts, among them U54 LM339, U55 MCP4728

Commit message: feat(hardware): frame-time inputs -- camera strobes back to GPIO26/27
Closes the gap camera-sync-change.md §3 opened. With the cameras free-running,
spec §12 item 1's justification for dropping exposure-active returns ("the Pi
triggers the cameras so frame times are known by construction") is false in
both halves. One FLIR ExposureActive strobe per camera group now returns on a
spare back-panel BNC and is timestamped in the same event stream as everything
else.

WHY A COMPARATOR AND NOT THIS BOARD'S USUAL INBOUND BUFFER. The strobe's best
published low is 0.87 V against SN74LVC541A's 0.8 V V_IL max -- a SILENT 70 mV
miss, on a signal that looks perfectly correct on a scope. A comparator is also
the only option here whose margin is a design choice rather than a datasheet
coincidence, which matters because FLIR label the whole table "values are for
reference only".

WHY +12V AND NOT +5V. The LM339's input common-mode ceiling is V+ - 1.5V to
V+ - 2.0V. The strobe's HIGH is 5.0 V (pulled up to +5V through 1k, FLIR's own
published row -- a stiffer pull-up makes V_low worse, not better). On a +5V
supply that ceiling is 3.0-3.5 V and the input sits above it, which is the
LM339's best-known failure mode. +12V/AGND matches U54 exactly.

GROUND DOMAINS, WHICH THE FIRST PASS GOT BACKWARDS. The pull-up sources from
+5V, whose return is DGND, so the shell net decides where 4.2 mA of switching
current flows: on AGND it would cross NT1, the single star tie, on every camera
frame; on DGND it never does. Shells, clamps and the threshold divider are
therefore DGND. V- stays AGND and does not enter the comparison -- both inputs
are DGND-referenced, so the offset is common-mode and cancels -- it sets only
the output LOW level, exactly as it already does for PD1_COMP/PD2_COMP/ACC_TRIG.

Tying the spare sections' inputs to DGND made U76 a SECOND AGND/DGND bridge
alongside NT1; check_breakout_power_netlist.py caught it. They go to AGND, this
part's own V-. A negative control now reproduce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
Parts:
- added C159, C160: 100nF, Capacitor_SMD:C_0603_1608Metric, symbol Device:C
- added D45, D46: BAT54S, Package_TO_SOT_SMD:SOT-23, symbol Diode:BAT54S
- added R209, R210, R213, R218: 10k, Resistor_SMD:R_0603_1608Metric, symbol Device:R
- added R211, R216: 100, Resistor_SMD:R_0603_1608Metric, symbol Device:R
- added R212, R217: 1k, Resistor_SMD:R_0603_1608Metric, symbol Device:R
- added R214, R219: 1M, Resistor_SMD:R_0603_1608Metric, symbol Device:R
- added R215, R220: 2.2k, Resistor_SMD:R_0603_1608Metric, symbol Device:R
- added U76: LM339, Package_SO:SOIC-14_3.9x8.7mm_P1.27mm, symbol Comparator:LM339
Connections:
- net +12V: now also C159.1, U76.3 (V+)
- net +3V3: now also R215.1, R220.1
- net AGND: now also C159.2, U76.11 (+), U76.12 (V-), U76.9 (+)
- new net +5V: D45.2 (K), D46.2 (K), R209.1, R212.1, R217.1
- new net CAM_FRAME_BEH: R219.1, R220.2, U76.1
- new net CAM_FRAME_BEH_BNC: R216.1
- new net CAM_FRAME_BEH_CLAMP: D46.3 (COM), R216.2, R217.2, R218.1
- new net CAM_FRAME_BEH_FB: R218.2, R219.2, U76.7 (+)
- new net CAM_FRAME_EYE: R214.1, R215.2, U76.2
- new net CAM_FRAME_EYE_BNC: R211.1
- new net CAM_FRAME_EYE_CLAMP: D45.3 (COM), R211.2, R212.2, R213.1
- new net CAM_FRAME_EYE_FB: R213.2, R214.2, U76.5 (+)
- new net CAM_FRAME_THR: C160.1, R209.2, R210.1, U76.10 (-), U76.4 (-), U76.6 (-), U76.8 (-)
- new net DGND: C160.2, D45.1 (A), D46.1 (A), R210.2
- no-connect marks 1 -> 3
Other:
- note added: "- The 1k pull-up sources from +5V, whose return is DGND. So the SHELL net picks"
- note added: "- V- stays AGND, like U54. It does not enter the COMPARISON: '+' and '-' are both"
- note added: "BY 70 mV, silently -- the buffer may simply never see a valid low on a signal that"
- note added: "CONNECTOR IN LAYOUT -- protection between panel and silicon has to be true in"
- note added: "CONNECTORS: spare ports J17B (pi-interface) and J6B (taskpc-digital), the only two"
- note added: "DGND-referenced, so an AGND-DGND offset is common-mode and cancels. What V-"
- note added: "FRAME-TIME INPUTS (2026-08-16) -- U76, the SECOND LM339 on this sheet, and the"
- note added: "MARGINS: 1.63 V low (0.87 V vs 2.50 V) and 2.50 V high (5.00 V vs 2.50 V). The"
- note added: "OUT OF BAND (U76/D45-D46/R209-R220/C159-C160), above the board-wide maxima, for the"
- note added: "SAME electrical interface -- ohDPI runs OpenIris -> Spinnaker -> FLIR BFS -- so"
- note added: "SOFTWARE MUST TIMESTAMP THE FALLING EDGE. ExposureActive asserts by pulling low and"
- note added: "Shells, BAT54S clamps and the 10k/10k threshold divider are therefore all DGND."
- note added: "The DAC note (VSS = AGND 'NOT DGND') is the SAME principle -- keep the threshold in"
- note added: "U76's other two sections are unused: inputs tied ('+' to AGND -- this part's own"
- note added: "V+ - 2.0V. The strobe's HIGH is 5.0 V (pulled up to +5V through 1k, FLIR's own"
- note added: "V-, and NOT DGND, which would make U76 a SECOND AGND/DGND bridge alongside NT1 and"
- note added: "WHY NOT STRAIGHT INTO A 74LVC541A INPUT LIKE EVERY OTHER DIGITAL INPUT HERE: the"
- note added: "WHY THE FRONT END IS DGND WHILE V- IS AGND -- NOT A CONTRADICTION:"
- note added: "WHY V+ = +12V AND NOT +5V: the LM339's input common-mode ceiling is V+ - 1.5V to"
- note added: "against DGND at a ~0.99 V V_IL. Identical to PD1_COMP/PD2_COMP/ACC_TRIG."
- note added: "allocated anyway. Its only effect is a constant sub-us offset on a 2 ms frame."
- note added: "and a 5.0 V input sits ABOVE it -- the LM339's best-known failure mode, an"
- note added: "anything from ~1.5 to ~3.5 V behaves identically, and all four MCP4728 channels are"
- note added: "break the board's single-point ground; '-' to the 2.50 V threshold) so nothing"
- note added: "carries a systematic error."
- note added: "copper, not only on a schematic sheet."
- note added: "floats, outputs no_connect with no pull-up, so they sink nothing. U76 therefore"
- note added: "inverted output. +12V puts the ceiling at 10.0 V. Same rail U54 already runs."
- note added: "is a design choice rather than a datasheet coincidence."
- note added: "looks perfectly correct on a scope. A comparator is the only option whose margin"
- note added: "one front end serves both. See hardware/breakout/frame-time-inputs.md."
- note added: "only DGND-referenced circuitry on it. Two FLIR Blackfly S ExposureActive strobes"
- note added: "published row: 0.87 V low / 5.0 V high / 4.2 mA). On +5V the ceiling is 3.0-3.5 V"
- note added: "return to GPIO26/27 (the last two non-PWM spares). Both camera groups are the"
- note added: "same reason R190 is -- see CHANNEL4_SERIES_REF."
- note added: "sets is the OUTPUT LOW (it is the common emitter): AGND + V_CEsat ~ 0.2 V, read"
- note added: "sits wholly in the AGND domain; only its passives touch DGND. Refdes here are minted"
- note added: "spare ports on the BACK face; their panel holes are already machined. Those sheets"
- note added: "strobe's best published low is 0.87 V and LVC541A's V_IL max is 0.8 V. It MISSES"
- note added: "that edge is actively driven by the opto transistor. The RISING edge is RC through"
- note added: "the other domain. It is not being contradicted here."
- note added: "the pull-up and varies with cable length, so pulse WIDTH measured off this signal"
- note added: "the signal's own domain -- reaching the other net because these signals arrive in"
- note added: "threshold needs no trimming and gets no DAC channel: the swing is 0.87-5.0 V, so"
- note added: "where 4.2 mA of switching current flows on every camera frame. On AGND it"
- note added: "wire centre and shell. THE 100R AND CLAMP ARE DRAWN HERE BUT MUST BE PLACED AT THE"
- note added: "would cross NT1, the board's single AGND/DGND star tie. On DGND it never does."
